Commit message: Fixing joints for gripper

File: gripper/urdf/gripper.urdf (robot description, URDF)
Before this commit: robot gripper, 9 links, 8 joints
Links:
- removed link gripper_base_link
- added link base_link, mass 0.080698; collision mesh filename=package://gripper/meshes/gripper_base_link.STL; visual mesh filename=package://gripper/meshes/gripper_base_link.STL
Joints:
- joint gripper_motor1_joint: parent gripper_base_link -> base_link
- joint gripper_motor2_joint: parent gripper_base_link -> base_link
- joint hand1_fingertip1_joint: axis 0 0 0 -> 0 0 1; limit lower=0 upper=0 effort=0 velocity=0 -> lower=-1 upper=1 effort=10 velocity=0.5; origin xyz=0.006 0.0072045 -0.057631 rpy=0 0.00089873 -1.5708 -> xyz=-0.0056 0.0877 0.0055 rpy=0 0 0
- joint hand1_fingertip2_joint: axis 0 0 0 -> 0 0 1; limit lower=0 upper=0 effort=0 velocity=0 -> lower=-1 upper=1 effort=10 velocity=0.5; origin xyz=0.038 0.0072769 -0.057346 rpy=3.1416 -0.4981 -1.5708 -> xyz=-0.0056 0.0877 -0.0055 rpy=0 0 0
- joint hand2_fingertip1_joint: axis 0 0 0 -> 0 0 1; limit lower=0 upper=0 effort=0 velocity=0 -> lower=-1 upper=1 effort=10 velocity=0.5; origin xyz=0.006 0.0072118 -0.057537 rpy=0 -0.15638 -1.5708 -> xyz=-0.0056 0.0877 0.0055 rpy=0 0 0
- joint hand2_fingertip2_joint: axis 0 0 0 -> 0 0 1; limit lower=0 upper=0 effort=0 velocity=0 -> lower=-1 upper=1 effort=10 velocity=0.5; origin xyz=0.038 0.0072072 -0.057573 rpy=3.1416 -0.095497 -1.5708 -> xyz=-0.0056 0.0877 -0.0055 rpy=0 0 0
- joint motor1_hand_joint: axis 0 0 0 -> 0 0 1; limit lower=0 upper=0 effort=0 velocity=0 -> lower=-1 upper=1 effort=10 velocity=0.5; origin xyz=-0.013151 0.029934 0.02235 rpy=1.5658 1.5708 0 -> xyz=0 0 0 rpy=0 0 0
- joint motor2_hand_joint: axis 0 0 0 -> 0 0 1; limit lower=0 upper=0 effort=0 velocity=0 -> lower=-1 upper=1 effort=10 velocity=0.5; origin xyz=-0.013151 0.029934 0.02235 rpy=1.5658 1.5708 0 -> xyz=0 0 0 rpy=0 0 0
