Commit message: Adding RGBD-cameras on arm

File: pmb2_robot/pmb2_description/urdf/arm/palbator_arm.urdf.xacro (robot description, xacro)
@@ -13,4 +13,5 @@
   <xacro:property name="Joint_Y_5_6" value="0.04" />
   <xacro:property name="Joint_Y_6_7" value="0.057" />
+  <xacro:property name="PI" value="3.14159"/>
   <xacro:macro name="palbator_arm" params="parent">
     <!-- <xacro:include filename="$(find cob_description)/gazebo/gazebo.urdf.xacro" /> -->
@@ -31,5 +32,5 @@
       </visual>
     </link>
-    <link name="palbator_arm_kinect" >
+    <link name="palbator_arm_kinect_link" >
       <inertial>
         <origin xyz="0 0 0" rpy="0 0 0"/>
@@ -184,5 +185,5 @@
     <joint name="palbator_arm_kinect_joint" type="fixed">
       <parent link="palbator_arm_column"/>
-      <child link="palbator_arm_kinect"/>
+      <child link="palbator_arm_kinect_link"/>
         <origin xyz="0.0 0.0 1.60" rpy="0 -0.3 0" />
         <axis xyz="0 0 1" />
@@ -333,4 +334,94 @@
       </actuator>
     </transmission>
+<!-- GAZEBO MATERIALS -->
+    <gazebo reference="palbator_arm_kinect_link">
+      <material>Gazebo/Black</material>
+    </gazebo>
+    <gazebo reference="palbator_arm_camera_link">
+      <material>Gazebo/Black</material>
+    </gazebo>
+<!-- GAZEBO PLUGINS -->
+  <gazebo reference="palbator_arm_camera_link">
+   <sensor name="palbator_arm_camera_link_camera" type="depth">
+     <update_rate>20</update_rate>
+     <camera>
+       <horizontal_fov>1.047198</horizontal_fov>
+       <image>
+         <width>640</width>
+         <height>480</height>
+         <format>R8G8B8</format>
+       </image>
+       <clip>
+         <near>0.05</near>
+         <far>5.0</far>
+       </clip>
+     </camera>
+     <plugin name="camera_plugin" filename="libgazebo_ros_openni_kinect.so">
+      <baseline>0.2</baseline>
+      <alwaysOn>true</alwaysOn>
+      <updateRate>20.0</updateRate>
+      <cameraName>camera_ir</cameraName>
+      <imageTopicName>/camera/color/image_raw</imageTopicName>
+      <cameraInfoTopicName>/camera/color/camera_info</cameraInfoTopicName>
+      <depthImageTopicName>/camera/depth/image_raw</depthImageTopicName>
+      <depthImageCameraInfoTopicName>/camera/depth/camera_info</depthImageCameraInfoTopicName>
+      <pointCloudTopicName>/camera/depth/points</pointCloudTopicName>
+      <frameName>palbator_arm_camera_link</frameName>
+      <pointCloudCutoff>0.5</pointCloudCutoff>
+      <pointCloudCutoffMax>3.0</pointCloudCutoffMax>
+      <distortionK1>0</distortionK1>
+      <distortionK2>0</distortionK2>
+      <distortionK3>0</distortionK3>
+      <distortionT1>0</distortionT1>
+      <distortionT2>0</distortionT2>
+      <CxPrime>0</CxPrime>
+      <Cx>0</Cx>
+      <Cy>0</Cy>
+      <focalLength>0</focalLength>
+      <hackBaseline>0</hackBaseline>
+     </plugin>
+   </sensor>
+  </gazebo>
+  <gazebo reference="palbator_arm_kinect_link">
+   <sensor name="palbator_arm_kinect_link_camera" type="depth">
+     <update_rate>20</update_rate>
+     <camera>
+       <horizontal_fov>1.047198</horizontal_fov>
+       <image>
+         <width>1920</width>
+         <height>1080</height>
+         <format>R8G8B8</format>
+       </image>
+       <clip>
+         <near>0.05</near>
+         <far>5.0</far>
+       </clip>
+     </camera>
+     <plugin name="camera_plugin" filename="libgazebo_ros_openni_kinect.so">
+      <baseline>0.2</baseline>
+      <alwaysOn>true</alwaysOn>
+      <updateRate>20.0</updateRate>
+      <cameraName>kinect_ir</cameraName>
+      <imageTopicName>/kinect/color/image_raw</imageTopicName>
+      <cameraInfoTopicName>/kinect/color/camera_info</cameraInfoTopicName>
+      <depthImageTopicName>/kinect/depth/image_raw</depthImageTopicName>
+      <depthImageCameraInfoTopicName>/kinect/depth/camera_info</depthImageCameraInfoTopicName>
+      <pointCloudTopicName>/kinect/depth/points</pointCloudTopicName>
+      <frameName>palbator_arm_kinect_link</frameName>
+      <pointCloudCutoff>0.5</pointCloudCutoff>
+      <pointCloudCutoffMax>3.0</pointCloudCutoffMax>
+      <distortionK1>0</distortionK1>
+      <distortionK2>0</distortionK2>
+      <distortionK3>0</distortionK3>
+      <distortionT1>0</distortionT1>
+      <distortionT2>0</distortionT2>
+      <CxPrime>0</CxPrime>
+      <Cx>0</Cx>
+      <Cy>0</Cy>
+      <focalLength>0</focalLength>
+      <hackBaseline>0</hackBaseline>
+     </plugin>
+   </sensor>
+  </gazebo>
   </xacro:macro>
 </robot>

Commit message: Fix kinect camera orientation

File: pmb2_robot/pmb2_description/urdf/arm/palbator_arm.urdf.xacro (robot description, xacro)
@@ -186,5 +186,5 @@
       <parent link="palbator_arm_column"/>
       <child link="palbator_arm_kinect_link"/>
-        <origin xyz="0.0 0.0 1.60" rpy="0 -0.3 0" />
+        <origin xyz="0.0 0.0 1.60" rpy="${PI} ${PI - 0.3} 0" />
         <axis xyz="0 0 1" />
     </joint>

Commit message: Adding gripper to robot xacro

File: pmb2_robot/pmb2_description/urdf/arm/palbator_arm.urdf.xacro (robot description, xacro)
@@ -14,4 +14,5 @@
   <xacro:property name="Joint_Y_6_7" value="0.057" />
   <xacro:property name="PI" value="3.14159"/>
+  <xacro:include filename="$(find pmb2_description)/urdf/gripper/gripper.urdf.xacro"/>
   <xacro:macro name="palbator_arm" params="parent">
     <!-- <xacro:include filename="$(find cob_description)/gazebo/gazebo.urdf.xacro" /> -->
@@ -135,4 +136,5 @@
       </visual>
     </link>
+<!--
     <link name="palbator_arm_wrist_link3" >
       <inertial>
@@ -151,4 +153,5 @@
       </visual>
     </link>
+    -->
   <!--
     <link name="grip_link" >
@@ -177,5 +180,5 @@
         </visual>
     </link>
-    <link name="palbator_arm_end_link" />
+    <!-- JOINTS -->
     <joint name="palbator_arm_to_${parent}_joint" type="fixed">
       <origin xyz="0 0 0.195" rpy="0 0 3.14" />
@@ -231,4 +234,5 @@
       <axis xyz="-1 0 0" />
     </joint>
+<!--
     <joint name="palbator_arm_wrist_3_joint" type="revolute">
       <parent link="palbator_arm_wrist_link2"/>
@@ -238,4 +242,5 @@
       <axis xyz="0 1 0" />
     </joint>
+-->
   <!--
     <joint name="grip_left_joint" type="fixed">
@@ -252,4 +257,5 @@
     </joint>
   -->
+<!--
     <joint name="palbator_arm_end_joint" type="fixed">
       <parent link="palbator_arm_wrist_link3"/>
@@ -258,4 +264,5 @@
       <axis xyz="0 0 0" />
     </joint>
+-->
     <joint name="palbator_arm_camera_joint" type="fixed">
       <parent link="palbator_arm_shoulder_link2"/>
@@ -264,4 +271,8 @@
       <axis xyz="0 0 0" />
     </joint>
+<!-- GRIPPER INCLUDE -->
+    <xacro:gripper parent="${name}_link">
+      <origin xyz="0 0.0275 0.012" rpy="0 0 0" />
+    </xacro:gripper>
     <transmission name="tran1">
       <type>SimpleTransmission</type>

Commit message: Update gripper pose in urdf

File: pmb2_robot/pmb2_description/urdf/arm/palbator_arm.urdf.xacro (robot description, xacro)
@@ -144,5 +144,4 @@
       </inertial>
       <visual>
-        <origin xyz="0 0.0275 0.012" rpy="0 0 0" />
         <geometry>
             <box size="0.13 0.045 0.06"/>
@@ -331,14 +330,4 @@
       </joint>
       <actuator name="motor6">
-        <hardwareInterface>hardware_interface/EffortJointInterface</hardwareInterface>
-        <mechanicalReduction>1</mechanicalReduction>
-      </actuator>
-    </transmission>
-    <transmission name="tran7">
-      <type>SimpleTransmission</type>
-      <joint name="palbator_arm_wrist_3_joint">
-        <hardwareInterface>hardware_interface/EffortJointInterface</hardwareInterface>
-      </joint>
-      <actuator name="motor7">
         <hardwareInterface>hardware_interface/EffortJointInterface</hardwareInterface>
         <mechanicalReduction>1</mechanicalReduction>

File: pmb2_robot/pmb2_description/urdf/gripper/gripper.urdf.xacro (robot description, xacro)
@@ -2,4 +2,5 @@
 <robot xmlns:xacro="http://ros.org/wiki/xacro">
   <xacro:macro name="gripper" params="parent *origin">
+  <xacro:property name="Joint_Y_6_7" value="0.057" />
     <!-- LINKS -->
     <link name="gripper_base_link">
@@ -16,5 +17,5 @@
       </inertial>
       <visual>
-        <origin xyz="0 0 0" rpy="0 0 0" />
+        <origin xyz="0 0.0275 0.012" rpy="0 0 0" />
         <geometry>
           <mesh filename="package://pmb2_description/meshes/gripper/gripper_base_link.STL" />

Commit message: Re-align gripper

File: pmb2_robot/pmb2_description/urdf/arm/palbator_arm.urdf.xacro (robot description, xacro)
@@ -44,6 +44,6 @@
         </geometry>
           <origin xyz="0 0 0" rpy="0 0 0"/>
-        <material name="Cyan">
-          <color rgba="0 1.0 1.0 1.0"/>
+        <material name="Black">
+          <color rgba="0 0 0 1.0"/>
         </material>
       </visual>
@@ -102,5 +102,5 @@
             <box size="0.05 ${Joint_Y_4_5} 0.05"/>
         </geometry>
-        <material name="Cyan">
+      <material name="Cyan">
         <color rgba="0 1.0 1.0 1.0"/>
       </material>
@@ -176,4 +176,7 @@
               <box size="0.03 0.18 0.02"/>
           </geometry>
+          <material name="Black">
+            <color rgba="0 0 0 1.0"/>
+          </material>
             <origin xyz="0 0 0" rpy="0 0 0"/>
         </visual>

File: pmb2_robot/pmb2_description/urdf/gripper/gripper.urdf.xacro (robot description, xacro)
@@ -266,5 +266,5 @@
     </joint>
     <joint name="gripper_motor1_joint" type="fixed">
-      <origin xyz="0.0448 0.025822 -0.022247" rpy="0 0 0" />
+      <origin xyz="0.0448 0.053322 -0.010247" rpy="0 0 0" />
       <parent link="gripper_base_link" />
       <child link="motor1_link" />
@@ -294,5 +294,5 @@
     </joint>
     <joint name="gripper_motor2_joint" type="fixed">
-      <origin xyz="-0.0448 0.021922 -0.022197" rpy="-3.1416 0 3.1416" />
+      <origin xyz="-0.0448 0.053322 -0.010247" rpy="-3.1416 0 3.1416" />
       <parent link="gripper_base_link" />
       <child link="motor2_link" />

Commit message: Fix depth sensor orientation between gazebo & rviz

File: pmb2_robot/pmb2_description/urdf/arm/palbator_arm.urdf.xacro (robot description, xacro)
@@ -273,4 +273,17 @@
       <axis xyz="0 0 0" />
     </joint>
+  <!-- Empty camera joint for fixing wrong depth sensor orientation -->
+  <joint name="camera_depth_joint" type="fixed">
+    <origin xyz="0 0 0" rpy="${-PI/2} 0 ${-PI/2} "/>
+    <parent link="palbator_arm_camera_link"/>
+    <child link="camera_depth_link"/>
+  </joint>
+  <link name="camera_depth_link"></link>
+  <joint name="kinect_depth_joint" type="fixed">
+    <origin xyz="0 0 0" rpy="${-PI/2} 0 ${-PI/2} "/>
+    <parent link="palbator_arm_kinect_link"/>
+    <child link="kinect_depth_link"/>
+  </joint>
+  <link name="kinect_depth_link"></link>
 <!-- GRIPPER INCLUDE -->
     <xacro:gripper parent="${name}_link">
@@ -370,5 +383,5 @@
       <depthImageCameraInfoTopicName>/camera/depth/camera_info</depthImageCameraInfoTopicName>
       <pointCloudTopicName>/camera/depth/points</pointCloudTopicName>
-      <frameName>palbator_arm_camera_link</frameName>
+      <frameName>camera_depth_link</frameName>
       <pointCloudCutoff>0.5</pointCloudCutoff>
       <pointCloudCutoffMax>3.0</pointCloudCutoffMax>
@@ -411,5 +424,5 @@
       <depthImageCameraInfoTopicName>/kinect/depth/camera_info</depthImageCameraInfoTopicName>
       <pointCloudTopicName>/kinect/depth/points</pointCloudTopicName>
-      <frameName>palbator_arm_kinect_link</frameName>
+      <frameName>kinect_depth_link</frameName>
       <pointCloudCutoff>0.5</pointCloudCutoff>
       <pointCloudCutoffMax>3.0</pointCloudCutoffMax>

Commit message: Last version URDF without gripper + linked moveit. From now until a gripper improvement, this URDF version will be used

File: pmb2_robot/pmb2_description/urdf/arm/palbator_arm.urdf.xacro (robot description, xacro)
@@ -14,5 +14,5 @@
   <xacro:property name="Joint_Y_6_7" value="0.057" />
   <xacro:property name="PI" value="3.14159"/>
-  <xacro:include filename="$(find pmb2_description)/urdf/gripper/gripper.urdf.xacro"/>
+  <!-- <xacro:include filename="$(find pmb2_description)/urdf/gripper/gripper.urdf.xacro"/> -->
   <xacro:macro name="palbator_arm" params="parent">
     <!-- <xacro:include filename="$(find cob_description)/gazebo/gazebo.urdf.xacro" /> -->
@@ -136,5 +136,4 @@
       </visual>
     </link>
-<!--
     <link name="palbator_arm_wrist_link3" >
       <inertial>
@@ -152,5 +151,5 @@
       </visual>
     </link>
-    -->
+    <link name="palbator_arm_end_link" />
   <!--
     <link name="grip_link" >
@@ -236,5 +235,4 @@
       <axis xyz="-1 0 0" />
     </joint>
-<!--
     <joint name="palbator_arm_wrist_3_joint" type="revolute">
       <parent link="palbator_arm_wrist_link2"/>
@@ -244,5 +242,4 @@
       <axis xyz="0 1 0" />
     </joint>
--->
   <!--
     <joint name="grip_left_joint" type="fixed">
@@ -259,5 +256,4 @@
     </joint>
   -->
-<!--
     <joint name="palbator_arm_end_joint" type="fixed">
       <parent link="palbator_arm_wrist_link3"/>
@@ -266,5 +262,4 @@
       <axis xyz="0 0 0" />
     </joint>
--->
     <joint name="palbator_arm_camera_joint" type="fixed">
       <parent link="palbator_arm_shoulder_link2"/>
@@ -273,21 +268,21 @@
       <axis xyz="0 0 0" />
     </joint>
-  <!-- Empty camera joint for fixing wrong depth sensor orientation -->
-  <joint name="camera_depth_joint" type="fixed">
-    <origin xyz="0 0 0" rpy="${-PI/2} 0 ${-PI/2} "/>
-    <parent link="palbator_arm_camera_link"/>
-    <child link="camera_depth_link"/>
-  </joint>
-  <link name="camera_depth_link"></link>
-  <joint name="kinect_depth_joint" type="fixed">
-    <origin xyz="0 0 0" rpy="${-PI/2} 0 ${-PI/2} "/>
-    <parent link="palbator_arm_kinect_link"/>
-    <child link="kinect_depth_link"/>
-  </joint>
-  <link name="kinect_depth_link"></link>
+    <!-- Empty camera joint for fixing wrong depth sensor orientation -->
+    <joint name="camera_depth_joint" type="fixed">
+      <origin xyz="0 0 0" rpy="${-PI/2} 0 ${-PI/2} "/>
+      <parent link="palbator_arm_camera_link"/>
+      <child link="camera_depth_link"/>
+    </joint>
+    <link name="camera_depth_link"></link>
+    <joint name="kinect_depth_joint" type="fixed">
+      <origin xyz="0 0 0" rpy="${-PI/2} 0 ${-PI/2} "/>
+      <parent link="palbator_arm_kinect_link"/>
+      <child link="kinect_depth_link"/>
+    </joint>
+    <link name="kinect_depth_link"></link>
 <!-- GRIPPER INCLUDE -->
-    <xacro:gripper parent="${name}_link">
+    <!-- <xacro:gripper parent="${name}_link">
       <origin xyz="0 0.0275 0.012" rpy="0 0 0" />
-    </xacro:gripper>
+    </xacro:gripper> -->
     <transmission name="tran1">
       <type>SimpleTransmission</type>
@@ -346,4 +341,14 @@
       </joint>
       <actuator name="motor6">
+        <hardwareInterface>hardware_interface/EffortJointInterface</hardwareInterface>
+        <mechanicalReduction>1</mechanicalReduction>
+      </actuator>
+    </transmission>
+    <transmission name="tran7">
+      <type>SimpleTransmission</type>
+      <joint name="palbator_arm_wrist_3_joint">
+        <hardwareInterface>hardware_interface/EffortJointInterface</hardwareInterface>
+      </joint>
+      <actuator name="motor7">
         <hardwareInterface>hardware_interface/EffortJointInterface</hardwareInterface>
         <mechanicalReduction>1</mechanicalReduction>

File: pmb2_robot/pmb2_description/urdf/arm/palbator_arm_with_gripper.urdf.xacro (robot description, xacro)
@@ -14,5 +14,5 @@
   <xacro:property name="Joint_Y_6_7" value="0.057" />
   <xacro:property name="PI" value="3.14159"/>
-  <!-- <xacro:include filename="$(find pmb2_description)/urdf/gripper/gripper.urdf.xacro"/> -->
+  <xacro:include filename="$(find pmb2_description)/urdf/gripper/gripper.urdf.xacro"/>
   <xacro:macro name="palbator_arm" params="parent">
     <!-- <xacro:include filename="$(find cob_description)/gazebo/gazebo.urdf.xacro" /> -->
@@ -136,4 +136,5 @@
       </visual>
     </link>
+<!--
     <link name="palbator_arm_wrist_link3" >
       <inertial>
@@ -151,5 +152,5 @@
       </visual>
     </link>
-    <link name="palbator_arm_end_link" />
+    -->
   <!--
     <link name="grip_link" >
@@ -204,5 +205,5 @@
       <child link="palbator_arm_shoulder_link1"/>
       <origin xyz="0 0 0" rpy="0 0 0" />
-      <limit effort="100" velocity="0.3" lower="-1.22" upper="1.22" />
+      <limit effort="1000" velocity="0.3" lower="-1.22" upper="1.22" />
       <axis xyz="0 0 1" />
     </joint>
@@ -218,5 +219,5 @@
       <child link="palbator_arm_shoulder_link3"/>
       <origin xyz="0 ${Joint_Y_3_4} 0" rpy="0 0 0" />
-      <limit effort="100" velocity="0.3" lower="-1.17" upper="1.6" />
+      <limit effort="1000" velocity="0.3" lower="-1.17" upper="1.6" />
       <axis xyz="-1 0 0" />
     </joint>
@@ -225,5 +226,5 @@
       <child link="palbator_arm_wrist_link1"/>
       <origin xyz="0 ${Joint_Y_4_5} 0" rpy="0 0 0" />
-      <limit effort="100" velocity="0.3" lower="-3.14" upper="3.14" />
+      <limit effort="1000" velocity="0.3" lower="-3.14" upper="3.14" />
       <axis xyz="0 1 0" />
     </joint>
@@ -232,7 +233,8 @@
       <child link="palbator_arm_wrist_link2"/>
       <origin xyz="0 ${Joint_Y_5_6} 0" rpy="0 0 0" />
-      <limit effort="100" velocity="0.3" lower="-1.5" upper="2.0" />
+      <limit effort="1000" velocity="0.3" lower="-1.5" upper="2.0" />
       <axis xyz="-1 0 0" />
     </joint>
+<!--
     <joint name="palbator_arm_wrist_3_joint" type="revolute">
       <parent link="palbator_arm_wrist_link2"/>
@@ -242,4 +244,5 @@
       <axis xyz="0 1 0" />
     </joint>
+-->
   <!--
     <joint name="grip_left_joint" type="fixed">
@@ -256,4 +259,5 @@
     </joint>
   -->
+<!--
     <joint name="palbator_arm_end_joint" type="fixed">
       <parent link="palbator_arm_wrist_link3"/>
@@ -262,4 +266,5 @@
       <axis xyz="0 0 0" />
     </joint>
+-->
     <joint name="palbator_arm_camera_joint" type="fixed">
       <parent link="palbator_arm_shoulder_link2"/>
@@ -268,8 +273,21 @@
       <axis xyz="0 0 0" />
     </joint>
+  <!-- Empty camera joint for fixing wrong depth sensor orientation -->
+  <joint name="camera_depth_joint" type="fixed">
+    <origin xyz="0 0 0" rpy="${-PI/2} 0 ${-PI/2} "/>
+    <parent link="palbator_arm_camera_link"/>
+    <child link="camera_depth_link"/>
+  </joint>
+  <link name="camera_depth_link"></link>
+  <joint name="kinect_depth_joint" type="fixed">
+    <origin xyz="0 0 0" rpy="${-PI/2} 0 ${-PI/2} "/>
+    <parent link="palbator_arm_kinect_link"/>
+    <child link="kinect_depth_link"/>
+  </joint>
+  <link name="kinect_depth_link"></link>
 <!-- GRIPPER INCLUDE -->
-    <!-- <xacro:gripper parent="${name}_link">
+    <xacro:gripper parent="${name}_link">
       <origin xyz="0 0.0275 0.012" rpy="0 0 0" />
-    </xacro:gripper> -->
+    </xacro:gripper>
     <transmission name="tran1">
       <type>SimpleTransmission</type>
@@ -328,14 +346,4 @@
       </joint>
       <actuator name="motor6">
-        <hardwareInterface>hardware_interface/EffortJointInterface</hardwareInterface>
-        <mechanicalReduction>1</mechanicalReduction>
-      </actuator>
-    </transmission>
-    <transmission name="tran7">
-      <type>SimpleTransmission</type>
-      <joint name="palbator_arm_wrist_3_joint">
-        <hardwareInterface>hardware_interface/EffortJointInterface</hardwareInterface>
-      </joint>
-      <actuator name="motor7">
         <hardwareInterface>hardware_interface/EffortJointInterface</hardwareInterface>
         <mechanicalReduction>1</mechanicalReduction>
@@ -375,5 +383,5 @@
       <depthImageCameraInfoTopicName>/camera/depth/camera_info</depthImageCameraInfoTopicName>
       <pointCloudTopicName>/camera/depth/points</pointCloudTopicName>
-      <frameName>palbator_arm_camera_link</frameName>
+      <frameName>camera_depth_link</frameName>
       <pointCloudCutoff>0.5</pointCloudCutoff>
       <pointCloudCutoffMax>3.0</pointCloudCutoffMax>
@@ -416,5 +424,5 @@
       <depthImageCameraInfoTopicName>/kinect/depth/camera_info</depthImageCameraInfoTopicName>
       <pointCloudTopicName>/kinect/depth/points</pointCloudTopicName>
-      <frameName>palbator_arm_kinect_link</frameName>
+      <frameName>kinect_depth_link</frameName>
       <pointCloudCutoff>0.5</pointCloudCutoff>
       <pointCloudCutoffMax>3.0</pointCloudCutoffMax>
