Commit message: update controllers, update column urdf

File: pmb2_robot/pmb2_description/urdf/arm/palbator_arm_with_gripper.urdf.xacro (robot description, xacro)
@@ -197,6 +197,6 @@
       <parent link="palbator_arm_column"/>
       <child link="palbator_arm_column_link"/>
-      <origin xyz="0 0.1 0" rpy="0 0 0" />
-      <limit effort="1000" velocity="0.3" lower="0.35" upper="1.35" />
+      <origin xyz="0 0.1 0.35" rpy="0 0 0" />
+      <limit effort="1000" velocity="0.3" lower="0" upper="1" />
       <axis xyz="0 0 1" />
     </joint>

Commit message: add face_screen

File: pmb2_robot/pmb2_description/urdf/arm/palbator_arm_with_gripper.urdf.xacro (robot description, xacro)
@@ -15,4 +15,5 @@
   <xacro:property name="PI" value="3.14159"/>
   <xacro:include filename="$(find pmb2_description)/urdf/gripper/gripper.urdf.xacro"/>
+  <xacro:include filename="$(find pmb2_description)/urdf/display/face_screen.urdf.xacro"/>
   <xacro:macro name="palbator_arm" params="parent">
     <!-- <xacro:include filename="$(find cob_description)/gazebo/gazebo.urdf.xacro" /> -->
@@ -191,5 +192,5 @@
       <parent link="palbator_arm_column"/>
       <child link="palbator_arm_kinect_link"/>
-        <origin xyz="0.0 0.0 1.60" rpy="${PI} ${PI - 0.3} 0" />
+        <origin xyz="-0.022 0.0 1.60" rpy="${PI} ${PI - 0.3} 0" />
         <axis xyz="0 0 1" />
     </joint>
@@ -290,4 +291,7 @@
       <origin xyz="0 0.0275 0.012" rpy="0 0 0" />
     </xacro:gripper>
+    <xacro:face_screen parent="${name}_link">
+      <origin xyz="0 0 0" rpy="0 0 0" />
+    </xacro:face_screen>
     <transmission name="tran1">
       <type>SimpleTransmission</type>

Commit message: Add logo + face texture(logo for the moment...) + real screen HRI

File: pmb2_robot/pmb2_description/urdf/arm/palbator_arm_with_gripper.urdf.xacro (robot description, xacro)
@@ -16,4 +16,6 @@
   <xacro:include filename="$(find pmb2_description)/urdf/gripper/gripper.urdf.xacro"/>
   <xacro:include filename="$(find pmb2_description)/urdf/display/face_screen.urdf.xacro"/>
+  <xacro:include filename="$(find pmb2_description)/urdf/display/hri_screen.urdf.xacro"/>
+  <xacro:include filename="$(find pmb2_description)/urdf/display/logos.urdf.xacro"/>
   <xacro:macro name="palbator_arm" params="parent">
     <!-- <xacro:include filename="$(find cob_description)/gazebo/gazebo.urdf.xacro" /> -->
@@ -287,11 +289,18 @@
   </joint>
   <link name="kinect_depth_link"></link>
+<!-- SCREENS INCLUDE -->
+    <xacro:face_screen parent="${name}_link">
+      <origin xyz="0 0 0" rpy="0 0 0" />
+    </xacro:face_screen>
+    <xacro:hri_screen parent="${name}_link">
+      <origin xyz="0 0 0" rpy="0 0 0" />
+    </xacro:hri_screen>
+    <xacro:logos parent="${name}_link">
+      <origin xyz="0 0 0" rpy="0 0 0" />
+    </xacro:logos>
 <!-- GRIPPER INCLUDE -->
     <xacro:gripper parent="${name}_link">
       <origin xyz="0 0.0275 0.012" rpy="0 0 0" />
     </xacro:gripper>
-    <xacro:face_screen parent="${name}_link">
-      <origin xyz="0 0 0" rpy="0 0 0" />
-    </xacro:face_screen>
     <transmission name="tran1">
       <type>SimpleTransmission</type>

File: pmb2_robot/pmb2_description/urdf/display/face_screen.urdf.xacro (robot description, xacro)
@@ -10,9 +10,6 @@
       <visual>
         <geometry>
-            <box size="0.01 0.18 0.12"/>
+            <box size="0.20 0.12 0.01"/>
         </geometry>
-        <!--<geometry>
-          <mesh filename="package://pmb2_description/meshes/display/face_screen.dae" scale="0.001 0.001 0.001"/>
-        </geometry>  -->
           <origin xyz="0 0 0" rpy="0 0 0"/>
         <material name="White">
@@ -21,11 +18,41 @@
       </visual>
     </link>
+    <link name="face_screen_display_link" >
+      <inertial>
+        <origin xyz="0 0 0" rpy="0 0 0"/>
+        <mass value="0.00001"/>
+        <inertia ixx="0.000001" ixy="0.0000001" ixz="0.0000001" iyy="0.0000001" iyz="0.0000001" izz="0.0000001"/>
+      </inertial>
+      <visual>
+        <geometry>
+          <mesh filename="package://pmb2_description/meshes/display/cpe-hand.dae" scale="0.1 0.06 100"/>
+        </geometry>
+      </visual>
+    </link>
     <!-- JOINTS -->
     <joint name="palbator_arm_face_screen_joint" type="fixed">
       <parent link="palbator_arm_column"/>
       <child link="face_screen_link"/>
-        <origin xyz="-0.04 0.0 1.505" rpy="0 0 0" />
+        <origin xyz="-0.04 0.0 1.505" rpy="1.57 0 -1.57" />
         <axis xyz="0 0 1" />
     </joint>
+    <joint name="face_screen_display_joint" type="fixed">
+      <parent link="face_screen_link"/>
+      <child link="face_screen_display_link"/>
+        <origin xyz="0 0 0.0051" rpy="0 0 0" />
+        <axis xyz="0 0 1" />
+    </joint>
+    <!-- GAZEBO PLUGINS -->
+<!--
+    <gazebo reference="face_screen_link">
+      <visual>
+        <plugin name="display_video_controller" filename="libgazebo_ros_video.so">
+          <topicName>/screen/face</topicName>
+          <height>120</height>
+          <width>180</width>
+        </plugin>
+      </visual>
+    </gazebo>
+-->
   </xacro:macro>
 </robot>

Commit message: add cart + camera holder + new gazebo colors

File: pmb2_robot/pmb2_description/urdf/arm/palbator_arm_with_gripper.urdf.xacro (robot description, xacro)
@@ -65,4 +65,100 @@
       </visual>
     </link>
+    <link name="cart_1_link" >
+      <inertial>
+        <origin xyz="0 0 0" rpy="0 0 0" />
+        <mass value="0.002"/>
+        <inertia ixx="0.001" ixy="0" ixz="0" iyy="0.001" iyz="0" izz="0.001"/>
+      </inertial>
+      <visual>
+        <origin xyz="0 0 0" rpy="0 0 0" />
+        <geometry>
+            <box size="0.02 0.14 0.08"/>
+        </geometry>
+        <material name="black">
+          <color rgba="0 0 0 1.0"/>
+        </material>
+      </visual>
+    </link>
+    <link name="cart_2_link" >
+      <inertial>
+        <origin xyz="0 0 0" rpy="0 0 0" />
+        <mass value="0.002"/>
+        <inertia ixx="0.001" ixy="0" ixz="0" iyy="0.001" iyz="0" izz="0.001"/>
+      </inertial>
+      <visual>
+        <origin xyz="0 0 0" rpy="0 0 0" />
+        <geometry>
+            <box size="0.02 0.14 0.08"/>
+        </geometry>
+        <material name="black">
+          <color rgba="0 0 0 1.0"/>
+        </material>
+      </visual>
+    </link>
+    <link name="cart_3_link" >
+      <inertial>
+        <origin xyz="0 0 0" rpy="0 0 0" />
+        <mass value="0.002"/>
+        <inertia ixx="0.001" ixy="0" ixz="0" iyy="0.001" iyz="0" izz="0.001"/>
+      </inertial>
+      <visual>
+        <origin xyz="0 0 0" rpy="0 0 0" />
+        <geometry>
+            <box size="0.10 0.02 0.16"/>
+        </geometry>
+        <material name="black">
+          <color rgba="0 0 0 1.0"/>
+        </material>
+      </visual>
+    </link>
+    <link name="cart_4_link" >
+      <inertial>
+        <origin xyz="0 0 0" rpy="0 0 0" />
+        <mass value="0.002"/>
+        <inertia ixx="0.001" ixy="0" ixz="0" iyy="0.001" iyz="0" izz="0.001"/>
+      </inertial>
+      <visual>
+        <origin xyz="0 0 0" rpy="0 0 0" />
+        <geometry>
+            <box size="0.12 0.02 0.08"/>
+        </geometry>
+        <material name="black">
+          <color rgba="0 0 0 1.0"/>
+        </material>
+      </visual>
+    </link>
+    <link name="cart_3A_link" >
+      <inertial>
+        <origin xyz="0 0 0" rpy="0 0 0" />
+        <mass value="0.002"/>
+        <inertia ixx="0.001" ixy="0" ixz="0" iyy="0.001" iyz="0" izz="0.001"/>
+      </inertial>
+      <visual>
+        <origin xyz="0 0 0" rpy="0 0 0" />
+        <geometry>
+            <box size="0.04 0.05 0.02"/>
+        </geometry>
+        <material name="black">
+          <color rgba="0 0 0 1.0"/>
+        </material>
+      </visual>
+    </link>
+    <link name="cart_3B_link" >
+      <inertial>
+        <origin xyz="0 0 0" rpy="0 0 0" />
+        <mass value="0.002"/>
+        <inertia ixx="0.001" ixy="0" ixz="0" iyy="0.001" iyz="0" izz="0.001"/>
+      </inertial>
+      <visual>
+        <origin xyz="0 0 0" rpy="0 0 0" />
+        <geometry>
+            <box size="0.04 0.05 0.02"/>
+        </geometry>
+        <material name="black">
+          <color rgba="0 0 0 1.0"/>
+        </material>
+      </visual>
+    </link>
     <link name="palbator_arm_shoulder_link1" >
       <inertial>
@@ -91,4 +187,30 @@
         <geometry>
             <box size="0.11 0.075 0.055"/>
+        </geometry>
+      </visual>
+    </link>
+    <link name="arm_cam_holder1_link" >
+      <inertial>
+          <origin xyz="0 0 0" rpy="0 0 0" />
+          <mass value="0.001"/>
+          <inertia ixx="0.001" ixy="0" ixz="0" iyy="0.001" iyz="0" izz="0.001"/>
+      </inertial>
+      <visual>
+        <origin xyz="0 0 0" rpy="0 0 0" />
+        <geometry>
+            <box size="0.06 0.04 0.02"/>
+        </geometry>
+      </visual>
+    </link>
+    <link name="arm_cam_holder2_link" >
+      <inertial>
+          <origin xyz="0 0 0" rpy="0 0 0" />
+          <mass value="0.001"/>
+          <inertia ixx="0.001" ixy="0" ixz="0" iyy="0.001" iyz="0" izz="0.001"/>
+      </inertial>
+      <visual>
+        <origin xyz="0 0 0" rpy="0 0 0" />
+        <geometry>
+            <box size="0.02 0.04 0.05"/>
         </geometry>
       </visual>
@@ -197,4 +319,40 @@
         <axis xyz="0 0 1" />
     </joint>
+    <joint name="cart_1_joint" type="fixed">
+      <parent link="palbator_arm_column_link"/>
+      <child link="cart_1_link"/>
+      <origin xyz="-0.06 -0.1 0.0" rpy="0 0 0" />
+      <axis xyz="0 0 1" />
+    </joint>
+    <joint name="cart_2_joint" type="fixed">
+      <parent link="palbator_arm_column_link"/>
+      <child link="cart_2_link"/>
+      <origin xyz="0.06 -0.1 0.0" rpy="0 0 0" />
+      <axis xyz="0 0 1" />
+    </joint>
+    <joint name="cart_3_joint" type="fixed">
+      <parent link="palbator_arm_column_link"/>
+      <child link="cart_3_link"/>
+      <origin xyz="0.0 -0.04 0.0" rpy="0 0 0" />
+      <axis xyz="0 0 1" />
+    </joint>
+    <joint name="cart_4_joint" type="fixed">
+      <parent link="palbator_arm_column_link"/>
+      <child link="cart_4_link"/>
+      <origin xyz="0.0 -0.16 0.0" rpy="0 0 0" />
+      <axis xyz="0 0 1" />
+    </joint>
+    <joint name="cart_3A_joint" type="fixed">
+      <parent link="palbator_arm_column_link"/>
+      <child link="cart_3A_link"/>
+      <origin xyz="0.0 -0.025 0.08" rpy="0 0 0" />
+      <axis xyz="0 0 1" />
+    </joint>
+    <joint name="cart_3B_joint" type="fixed">
+      <parent link="palbator_arm_column_link"/>
+      <child link="cart_3B_link"/>
+      <origin xyz="0.0 -0.025 -0.08" rpy="0 0 0" />
+      <axis xyz="0 0 1" />
+    </joint>
     <joint name="palbator_arm_column_joint" type="prismatic">
       <parent link="palbator_arm_column"/>
@@ -274,4 +432,16 @@
       <child link="palbator_arm_camera_link"/>
       <origin xyz="0.0 -0.05 0.20" rpy="0 0.5 1.57" />
+      <axis xyz="0 0 0" />
+    </joint>
+    <joint name="arm_cam_holder1_joint" type="fixed">
+      <parent link="palbator_arm_shoulder_link2"/>
+      <child link="arm_cam_holder1_link"/>
+      <origin xyz="0.0 -0.036 0.135" rpy="0 0 1.57" />
+      <axis xyz="0 0 0" />
+    </joint>
+    <joint name="arm_cam_holder2_joint" type="fixed">
+      <parent link="arm_cam_holder1_link"/>
+      <child link="arm_cam_holder2_link"/>
+      <origin xyz="-0.02 0 0.03" rpy="0 0 0" />
       <axis xyz="0 0 0" />
     </joint>
@@ -370,4 +540,22 @@
       <material>Gazebo/Black</material>
     </gazebo>
+  <gazebo reference="palbator_arm_column">
+    <material>Gazebo/DarkGrey</material>
+  </gazebo>
+  <gazebo reference="palbator_arm_shoulder_link1">
+    <material>Gazebo/Orange</material>
+  </gazebo>
+  <gazebo reference="palbator_arm_shoulder_link2">
+    <material>Gazebo/Orange</material>
+  </gazebo>
+  <gazebo reference="palbator_arm_shoulder_link3">
+    <material>Gazebo/Orange</material>
+  </gazebo>
+  <gazebo reference="palbator_arm_wrist_link1">
+    <material>Gazebo/Orange</material>
+  </gazebo>
+  <gazebo reference="palbator_arm_wrist_link2">
+    <material>Gazebo/Orange</material>
+  </gazebo>
 <!-- GAZEBO PLUGINS -->
   <gazebo reference="palbator_arm_camera_link">

File: pmb2_robot/pmb2_description/urdf/display/logos.urdf.xacro (robot description, xacro)
@@ -2,5 +2,4 @@
 <robot xmlns:xacro="http://ros.org/wiki/xacro">
   <xacro:macro name="logos" params="parent *origin">
-<!--
     <link name="logo_cpe_1" >
       <inertial>
@@ -11,9 +10,8 @@
       <visual>
         <geometry>
-          <mesh filename="package://pmb2_description/meshes/display/cpe-hand.dae" scale="0.04 0.025 1"/>
+          <mesh filename="package://pmb2_description/meshes/display/cpe-hand.dae" scale="0.07 0.04 1"/>
         </geometry>
       </visual>
     </link>
-    -->
     <link name="logo_lyontech_1" >
       <inertial>
@@ -113,12 +111,10 @@
     </link>
     <!-- JOINTS -->
-    <!--
     <joint name="logo_cpe_1_joint" type="fixed">
-      <parent link="palbator_arm_column"/>
+      <parent link="cart_1_link"/>
       <child link="logo_cpe_1"/>
-        <origin xyz="-0.041 0.0 1.2" rpy="1.57 0 -1.57" />
+        <origin xyz="-0.011 0.0 0.0" rpy="1.57 0 -1.57" />
         <axis xyz="0 0 1" />
     </joint>
--->
      <!-- LYONTECH -->
     <joint name="logo_lyontech_1_joint" type="fixed">

Commit message: Merge remote-tracking branch 'origin/upgrade_urdf' into dev_melodic_gripper

File: pmb2_robot/pmb2_description/urdf/arm/palbator_arm_with_gripper.urdf.xacro (robot description, xacro)
@@ -15,4 +15,7 @@
   <xacro:property name="PI" value="3.14159"/>
   <xacro:include filename="$(find pmb2_description)/urdf/gripper/gripper.urdf.xacro"/>
+  <xacro:include filename="$(find pmb2_description)/urdf/display/face_screen.urdf.xacro"/>
+  <xacro:include filename="$(find pmb2_description)/urdf/display/hri_screen.urdf.xacro"/>
+  <xacro:include filename="$(find pmb2_description)/urdf/display/logos.urdf.xacro"/>
   <xacro:macro name="palbator_arm" params="parent">
     <!-- <xacro:include filename="$(find cob_description)/gazebo/gazebo.urdf.xacro" /> -->
@@ -62,4 +65,100 @@
       </visual>
     </link>
+    <link name="cart_1_link" >
+      <inertial>
+        <origin xyz="0 0 0" rpy="0 0 0" />
+        <mass value="0.002"/>
+        <inertia ixx="0.001" ixy="0" ixz="0" iyy="0.001" iyz="0" izz="0.001"/>
+      </inertial>
+      <visual>
+        <origin xyz="0 0 0" rpy="0 0 0" />
+        <geometry>
+            <box size="0.02 0.14 0.08"/>
+        </geometry>
+        <material name="black">
+          <color rgba="0 0 0 1.0"/>
+        </material>
+      </visual>
+    </link>
+    <link name="cart_2_link" >
+      <inertial>
+        <origin xyz="0 0 0" rpy="0 0 0" />
+        <mass value="0.002"/>
+        <inertia ixx="0.001" ixy="0" ixz="0" iyy="0.001" iyz="0" izz="0.001"/>
+      </inertial>
+      <visual>
+        <origin xyz="0 0 0" rpy="0 0 0" />
+        <geometry>
+            <box size="0.02 0.14 0.08"/>
+        </geometry>
+        <material name="black">
+          <color rgba="0 0 0 1.0"/>
+        </material>
+      </visual>
+    </link>
+    <link name="cart_3_link" >
+      <inertial>
+        <origin xyz="0 0 0" rpy="0 0 0" />
+        <mass value="0.002"/>
+        <inertia ixx="0.001" ixy="0" ixz="0" iyy="0.001" iyz="0" izz="0.001"/>
+      </inertial>
+      <visual>
+        <origin xyz="0 0 0" rpy="0 0 0" />
+        <geometry>
+            <box size="0.10 0.02 0.16"/>
+        </geometry>
+        <material name="black">
+          <color rgba="0 0 0 1.0"/>
+        </material>
+      </visual>
+    </link>
+    <link name="cart_4_link" >
+      <inertial>
+        <origin xyz="0 0 0" rpy="0 0 0" />
+        <mass value="0.002"/>
+        <inertia ixx="0.001" ixy="0" ixz="0" iyy="0.001" iyz="0" izz="0.001"/>
+      </inertial>
+      <visual>
+        <origin xyz="0 0 0" rpy="0 0 0" />
+        <geometry>
+            <box size="0.12 0.02 0.08"/>
+        </geometry>
+        <material name="black">
+          <color rgba="0 0 0 1.0"/>
+        </material>
+      </visual>
+    </link>
+    <link name="cart_3A_link" >
+      <inertial>
+        <origin xyz="0 0 0" rpy="0 0 0" />
+        <mass value="0.002"/>
+        <inertia ixx="0.001" ixy="0" ixz="0" iyy="0.001" iyz="0" izz="0.001"/>
+      </inertial>
+      <visual>
+        <origin xyz="0 0 0" rpy="0 0 0" />
+        <geometry>
+            <box size="0.04 0.05 0.02"/>
+        </geometry>
+        <material name="black">
+          <color rgba="0 0 0 1.0"/>
+        </material>
+      </visual>
+    </link>
+    <link name="cart_3B_link" >
+      <inertial>
+        <origin xyz="0 0 0" rpy="0 0 0" />
+        <mass value="0.002"/>
+        <inertia ixx="0.001" ixy="0" ixz="0" iyy="0.001" iyz="0" izz="0.001"/>
+      </inertial>
+      <visual>
+        <origin xyz="0 0 0" rpy="0 0 0" />
+        <geometry>
+            <box size="0.04 0.05 0.02"/>
+        </geometry>
+        <material name="black">
+          <color rgba="0 0 0 1.0"/>
+        </material>
+      </visual>
+    </link>
     <link name="palbator_arm_shoulder_link1" >
       <inertial>
@@ -88,4 +187,30 @@
         <geometry>
             <box size="0.11 0.075 0.055"/>
+        </geometry>
+      </visual>
+    </link>
+    <link name="arm_cam_holder1_link" >
+      <inertial>
+          <origin xyz="0 0 0" rpy="0 0 0" />
+          <mass value="0.001"/>
+          <inertia ixx="0.001" ixy="0" ixz="0" iyy="0.001" iyz="0" izz="0.001"/>
+      </inertial>
+      <visual>
+        <origin xyz="0 0 0" rpy="0 0 0" />
+        <geometry>
+            <box size="0.06 0.04 0.02"/>
+        </geometry>
+      </visual>
+    </link>
+    <link name="arm_cam_holder2_link" >
+      <inertial>
+          <origin xyz="0 0 0" rpy="0 0 0" />
+          <mass value="0.001"/>
+          <inertia ixx="0.001" ixy="0" ixz="0" iyy="0.001" iyz="0" izz="0.001"/>
+      </inertial>
+      <visual>
+        <origin xyz="0 0 0" rpy="0 0 0" />
+        <geometry>
+            <box size="0.02 0.04 0.05"/>
         </geometry>
       </visual>
@@ -191,6 +316,42 @@
       <parent link="palbator_arm_column"/>
       <child link="palbator_arm_kinect_link"/>
-        <origin xyz="0.0 0.0 1.60" rpy="${PI} ${PI - 0.3} 0" />
+        <origin xyz="-0.022 0.0 1.60" rpy="${PI} ${PI - 0.3} 0" />
         <axis xyz="0 0 1" />
+    </joint>
+    <joint name="cart_1_joint" type="fixed">
+      <parent link="palbator_arm_column_link"/>
+      <child link="cart_1_link"/>
+      <origin xyz="-0.06 -0.1 0.0" rpy="0 0 0" />
+      <axis xyz="0 0 1" />
+    </joint>
+    <joint name="cart_2_joint" type="fixed">
+      <parent link="palbator_arm_column_link"/>
+      <child link="cart_2_link"/>
+      <origin xyz="0.06 -0.1 0.0" rpy="0 0 0" />
+      <axis xyz="0 0 1" />
+    </joint>
+    <joint name="cart_3_joint" type="fixed">
+      <parent link="palbator_arm_column_link"/>
+      <child link="cart_3_link"/>
+      <origin xyz="0.0 -0.04 0.0" rpy="0 0 0" />
+      <axis xyz="0 0 1" />
+    </joint>
+    <joint name="cart_4_joint" type="fixed">
+      <parent link="palbator_arm_column_link"/>
+      <child link="cart_4_link"/>
+      <origin xyz="0.0 -0.16 0.0" rpy="0 0 0" />
+      <axis xyz="0 0 1" />
+    </joint>
+    <joint name="cart_3A_joint" type="fixed">
+      <parent link="palbator_arm_column_link"/>
+      <child link="cart_3A_link"/>
+      <origin xyz="0.0 -0.025 0.08" rpy="0 0 0" />
+      <axis xyz="0 0 1" />
+    </joint>
+    <joint name="cart_3B_joint" type="fixed">
+      <parent link="palbator_arm_column_link"/>
+      <child link="cart_3B_link"/>
+      <origin xyz="0.0 -0.025 -0.08" rpy="0 0 0" />
+      <axis xyz="0 0 1" />
     </joint>
     <joint name="palbator_arm_column_joint" type="prismatic">
@@ -271,4 +432,16 @@
       <child link="palbator_arm_camera_link"/>
       <origin xyz="0.0 -0.05 0.20" rpy="0 0.5 1.57" />
+      <axis xyz="0 0 0" />
+    </joint>
+    <joint name="arm_cam_holder1_joint" type="fixed">
+      <parent link="palbator_arm_shoulder_link2"/>
+      <child link="arm_cam_holder1_link"/>
+      <origin xyz="0.0 -0.036 0.135" rpy="0 0 1.57" />
+      <axis xyz="0 0 0" />
+    </joint>
+    <joint name="arm_cam_holder2_joint" type="fixed">
+      <parent link="arm_cam_holder1_link"/>
+      <child link="arm_cam_holder2_link"/>
+      <origin xyz="-0.02 0 0.03" rpy="0 0 0" />
       <axis xyz="0 0 0" />
     </joint>
@@ -286,4 +459,14 @@
   </joint>
   <link name="kinect_depth_link"></link>
+<!-- SCREENS INCLUDE -->
+    <xacro:face_screen parent="${name}_link">
+      <origin xyz="0 0 0" rpy="0 0 0" />
+    </xacro:face_screen>
+    <xacro:hri_screen parent="${name}_link">
+      <origin xyz="0 0 0" rpy="0 0 0" />
+    </xacro:hri_screen>
+    <xacro:logos parent="${name}_link">
+      <origin xyz="0 0 0" rpy="0 0 0" />
+    </xacro:logos>
 <!-- GRIPPER INCLUDE -->
     <xacro:gripper parent="${name}_link">
@@ -357,4 +540,22 @@
       <material>Gazebo/Black</material>
     </gazebo>
+  <gazebo reference="palbator_arm_column">
+    <material>Gazebo/DarkGrey</material>
+  </gazebo>
+  <gazebo reference="palbator_arm_shoulder_link1">
+    <material>Gazebo/Orange</material>
+  </gazebo>
+  <gazebo reference="palbator_arm_shoulder_link2">
+    <material>Gazebo/Orange</material>
+  </gazebo>
+  <gazebo reference="palbator_arm_shoulder_link3">
+    <material>Gazebo/Orange</material>
+  </gazebo>
+  <gazebo reference="palbator_arm_wrist_link1">
+    <material>Gazebo/Orange</material>
+  </gazebo>
+  <gazebo reference="palbator_arm_wrist_link2">
+    <material>Gazebo/Orange</material>
+  </gazebo>
 <!-- GAZEBO PLUGINS -->
   <gazebo reference="palbator_arm_camera_link">

Commit message: update column range

File: pmb2_robot/pmb2_description/urdf/arm/palbator_arm_with_gripper.urdf.xacro (robot description, xacro)
@@ -358,5 +358,5 @@
       <parent link="palbator_arm_column"/>
       <child link="palbator_arm_column_link"/>
-      <origin xyz="0 0.1 0.35" rpy="0 0 0" />
+      <origin xyz="0 0.1 0.11" rpy="0 0 0" />
       <limit effort="1000" velocity="0.3" lower="0" upper="1" />
       <axis xyz="0 0 1" />
@@ -373,5 +373,5 @@
       <child link="palbator_arm_shoulder_link2"/>
       <origin xyz="0 ${Joint_Y_2_3} ${Joint_Z_2_3}" rpy="0 0 0" />
-      <limit effort="100" velocity="0.3" lower="-2.5" upper="2.27" />
+      <limit effort="1000" velocity="0.3" lower="-2.5" upper="2.27" />
       <axis xyz="0 0 -1" />
     </joint>
