Commit message: full logos (Lyontech + CPE) + Face on fake screen

File: pmb2_robot/pmb2_description/urdf/display/face_screen.urdf.xacro (robot description, xacro)
@@ -26,5 +26,5 @@
       <visual>
         <geometry>
-          <mesh filename="package://pmb2_description/meshes/display/cpe-hand.dae" scale="0.1 0.06 100"/>
+          <mesh filename="package://pmb2_description/meshes/display/PALbator_face.dae" scale="0.1 0.06 100"/>
         </geometry>
       </visual>

File: pmb2_robot/pmb2_description/urdf/display/logos.urdf.xacro (robot description, xacro)
@@ -2,4 +2,5 @@
 <robot xmlns:xacro="http://ros.org/wiki/xacro">
   <xacro:macro name="logos" params="parent *origin">
+<!--
     <link name="logo_cpe_1" >
       <inertial>
@@ -14,5 +15,103 @@
       </visual>
     </link>
+    -->
+    <link name="logo_lyontech_1" >
+      <inertial>
+        <origin xyz="0 0 0" rpy="0 0 0"/>
+        <mass value="0.00001"/>
+        <inertia ixx="0.000001" ixy="0.0000001" ixz="0.0000001" iyy="0.0000001" iyz="0.0000001" izz="0.0000001"/>
+      </inertial>
+      <visual>
+        <geometry>
+          <mesh filename="package://pmb2_description/meshes/display/lyontech.dae" scale="0.04 0.05 1"/>
+        </geometry>
+      </visual>
+    </link>
+    <link name="logo_lyontech_2" >
+      <inertial>
+        <origin xyz="0 0 0" rpy="0 0 0"/>
+        <mass value="0.00001"/>
+        <inertia ixx="0.000001" ixy="0.0000001" ixz="0.0000001" iyy="0.0000001" iyz="0.0000001" izz="0.0000001"/>
+      </inertial>
+      <visual>
+        <geometry>
+          <mesh filename="package://pmb2_description/meshes/display/lyontech.dae" scale="0.04 0.05 1"/>
+        </geometry>
+      </visual>
+    </link>
+    <link name="logo_lyontech_3" >
+      <inertial>
+        <origin xyz="0 0 0" rpy="0 0 0"/>
+        <mass value="0.00001"/>
+        <inertia ixx="0.000001" ixy="0.0000001" ixz="0.0000001" iyy="0.0000001" iyz="0.0000001" izz="0.0000001"/>
+      </inertial>
+      <visual>
+        <geometry>
+          <mesh filename="package://pmb2_description/meshes/display/lyontech.dae" scale="0.04 0.05 1"/>
+        </geometry>
+      </visual>
+    </link>
+    <link name="logo_lyontech_4" >
+      <inertial>
+        <origin xyz="0 0 0" rpy="0 0 0"/>
+        <mass value="0.00001"/>
+        <inertia ixx="0.000001" ixy="0.0000001" ixz="0.0000001" iyy="0.0000001" iyz="0.0000001" izz="0.0000001"/>
+      </inertial>
+      <visual>
+        <geometry>
+          <mesh filename="package://pmb2_description/meshes/display/lyontech.dae" scale="0.04 0.05 1"/>
+        </geometry>
+      </visual>
+    </link>
+    <link name="logo_palbator_cpe_1" >
+      <inertial>
+        <origin xyz="0 0 0" rpy="0 0 0"/>
+        <mass value="0.00001"/>
+        <inertia ixx="0.000001" ixy="0.0000001" ixz="0.0000001" iyy="0.0000001" iyz="0.0000001" izz="0.0000001"/>
+      </inertial>
+      <visual>
+        <geometry>
+          <mesh filename="package://pmb2_description/meshes/display/PALbator_cpe.dae" scale="0.04 0.04 1"/>
+        </geometry>
+      </visual>
+    </link>
+    <link name="logo_palbator_cpe_2" >
+      <inertial>
+        <origin xyz="0 0 0" rpy="0 0 0"/>
+        <mass value="0.00001"/>
+        <inertia ixx="0.000001" ixy="0.0000001" ixz="0.0000001" iyy="0.0000001" iyz="0.0000001" izz="0.0000001"/>
+      </inertial>
+      <visual>
+        <geometry>
+          <mesh filename="package://pmb2_description/meshes/display/PALbator_cpe.dae" scale="0.04 0.04 1"/>
+        </geometry>
+      </visual>
+    </link>
+    <link name="logo_palbator_cpe_3" >
+      <inertial>
+        <origin xyz="0 0 0" rpy="0 0 0"/>
+        <mass value="0.00001"/>
+        <inertia ixx="0.000001" ixy="0.0000001" ixz="0.0000001" iyy="0.0000001" iyz="0.0000001" izz="0.0000001"/>
+      </inertial>
+      <visual>
+        <geometry>
+          <mesh filename="package://pmb2_description/meshes/display/PALbator_cpe.dae" scale="0.04 0.04 1"/>
+        </geometry>
+      </visual>
+    </link>
+    <link name="logo_palbator_cpe_4" >
+      <inertial>
+        <origin xyz="0 0 0" rpy="0 0 0"/>
+        <mass value="0.00001"/>
+        <inertia ixx="0.000001" ixy="0.0000001" ixz="0.0000001" iyy="0.0000001" iyz="0.0000001" izz="0.0000001"/>
+      </inertial>
+      <visual>
+        <geometry>
+          <mesh filename="package://pmb2_description/meshes/display/PALbator_cpe.dae" scale="0.04 0.04 1"/>
+        </geometry>
+      </visual>
+    </link>
     <!-- JOINTS -->
+    <!--
     <joint name="logo_cpe_1_joint" type="fixed">
       <parent link="palbator_arm_column"/>
@@ -21,4 +120,55 @@
         <axis xyz="0 0 1" />
     </joint>
+-->
+     <!-- LYONTECH -->
+    <joint name="logo_lyontech_1_joint" type="fixed">
+      <parent link="palbator_arm_column"/>
+      <child link="logo_lyontech_1"/>
+        <origin xyz="-0.041 0.0 1.35" rpy="1.57 0 -1.57" />
+        <axis xyz="0 0 1" />
+    </joint>
+    <joint name="logo_lyontech_2_joint" type="fixed">
+      <parent link="palbator_arm_column"/>
+      <child link="logo_lyontech_2"/>
+        <origin xyz="0 -0.041 1.35" rpy="1.57 0 0" />
+        <axis xyz="0 0 1" />
+    </joint>
+    <joint name="logo_lyontech_3_joint" type="fixed">
+      <parent link="palbator_arm_column"/>
+      <child link="logo_lyontech_3"/>
+        <origin xyz="0 0.041 1.35" rpy="1.57 0 -3.14157" />
+        <axis xyz="0 0 1" />
+    </joint>
+    <joint name="logo_lyontech_4_joint" type="fixed">
+      <parent link="palbator_arm_column"/>
+      <child link="logo_lyontech_4"/>
+        <origin xyz="0.041 0.0 1.35" rpy="1.57 0 1.57" />
+        <axis xyz="0 0 1" />
+    </joint>
+    <!-- PALbator CPE -->
+    <joint name="logo_palbator_cpe_1_joint" type="fixed">
+      <parent link="palbator_arm_column"/>
+      <child link="logo_palbator_cpe_1"/>
+        <origin xyz="-0.041 0.0 1.25" rpy="1.57 0 -1.57" />
+        <axis xyz="0 0 1" />
+    </joint>
+    <joint name="logo_palbator_cpe_2_joint" type="fixed">
+      <parent link="palbator_arm_column"/>
+      <child link="logo_palbator_cpe_2"/>
+        <origin xyz="0 -0.041 1.25" rpy="1.57 0 0" />
+        <axis xyz="0 0 1" />
+    </joint>
+    <joint name="logo_palbator_cpe_3_joint" type="fixed">
+      <parent link="palbator_arm_column"/>
+      <child link="logo_palbator_cpe_3"/>
+        <origin xyz="0 0.041 1.25" rpy="1.57 0 -3.14157" />
+        <axis xyz="0 0 1" />
+    </joint>
+    <joint name="logo_palbator_cpe_4_joint" type="fixed">
+      <parent link="palbator_arm_column"/>
+      <child link="logo_palbator_cpe_4"/>
+        <origin xyz="0.041 0.0 1.25" rpy="1.57 0 1.57" />
+        <axis xyz="0 0 1" />
+    </joint>
   </xacro:macro>
 </robot>
