Commit message: add hri-screen holder

File: pmb2_robot/pmb2_description/urdf/display/hri_screen.urdf.xacro (robot description, xacro)
@@ -21,9 +21,119 @@
       </visual>
     </link>
+    <link name="column_back">
+      <inertial>
+        <origin xyz="0 0 0.75" rpy="0 0 0" />
+        <mass value="0.02"/>
+        <inertia ixx="0.01" ixy="0" ixz="0" iyy="0.01" iyz="0" izz="0.01"/>
+      </inertial>
+      <visual>
+        <origin xyz="0 0 0.75" rpy="0 0 0" />
+        <geometry>
+            <box size="0.02 0.04 1.5"/>
+        </geometry>
+        <material name="Gray_alu">
+          <color rgba="0.5 0.5 0.5 1.0"/>
+        </material>
+      </visual>
+    </link>
+    <link name="column_back_top">
+      <inertial>
+        <origin xyz="0 0 0" rpy="0 0 0" />
+        <mass value="0.002"/>
+        <inertia ixx="0.001" ixy="0" ixz="0" iyy="0.001" iyz="0" izz="0.001"/>
+      </inertial>
+      <visual>
+        <origin xyz="0 0 0" rpy="0 0 0" />
+        <geometry>
+            <box size="0.05 0.04 0.01"/>
+        </geometry>
+        <material name="Gray_alu">
+          <color rgba="0.5 0.5 0.5 1.0"/>
+        </material>
+      </visual>
+    </link>
+    <link name="column_back_screen_holder_1">
+      <inertial>
+        <origin xyz="0 0 0" rpy="0 0 0" />
+        <mass value="0.002"/>
+        <inertia ixx="0.001" ixy="0" ixz="0" iyy="0.001" iyz="0" izz="0.001"/>
+      </inertial>
+      <visual>
+        <origin xyz="0 0 0" rpy="0 0 0" />
+        <geometry>
+            <box size="0.02 0.12 0.04"/>
+        </geometry>
+        <material name="black">
+          <color rgba="0 0 0 1.0"/>
+        </material>
+      </visual>
+    </link>
+    <link name="column_back_screen_holder_2">
+      <inertial>
+        <origin xyz="0 0 0" rpy="0 0 0" />
+        <mass value="0.002"/>
+        <inertia ixx="0.001" ixy="0" ixz="0" iyy="0.001" iyz="0" izz="0.001"/>
+      </inertial>
+      <visual>
+        <origin xyz="0 0 0" rpy="0 0 0" />
+        <geometry>
+            <box size="0.24 0.02 0.04"/>
+        </geometry>
+        <material name="black">
+          <color rgba="0 0 0 1.0"/>
+        </material>
+      </visual>
+    </link>
+    <link name="column_back_screen_holder_3">
+      <inertial>
+        <origin xyz="0 0 0" rpy="0 0 0" />
+        <mass value="0.002"/>
+        <inertia ixx="0.001" ixy="0" ixz="0" iyy="0.001" iyz="0" izz="0.001"/>
+      </inertial>
+      <visual>
+        <origin xyz="0 0 0" rpy="0 0 0" />
+        <geometry>
+            <box size="0.02 -0.14 0.04"/>
+        </geometry>
+        <material name="black">
+          <color rgba="0 0 0 1.0"/>
+        </material>
+      </visual>
+    </link>
     <!-- JOINTS -->
+    <joint name="column_back_joint" type="fixed">
+      <parent link="palbator_arm_column"/>
+      <child link="column_back"/>
+        <origin xyz="0.1 0.0 0.0" rpy="0 0 0" />
+        <axis xyz="0 0 1" />
+    </joint>
+    <joint name="column_back_top_joint" type="fixed">
+      <parent link="column_back"/>
+      <child link="column_back_top"/>
+        <origin xyz="-0.035 0.0 1.495" rpy="0 0 0" />
+        <axis xyz="0 0 1" />
+    </joint>
+    <joint name="column_back_screen_holder_1_joint" type="fixed">
+      <parent link="column_back"/>
+      <child link="column_back_screen_holder_1"/>
+        <origin xyz="0 -0.07 0.8" rpy="0 0 0" />
+        <axis xyz="0 0 1" />
+    </joint>
+    <joint name="column_back_screen_holder_2_joint" type="fixed">
+      <parent link="column_back_screen_holder_1"/>
+      <child link="column_back_screen_holder_2"/>
+        <origin xyz="-0.11 -0.07 0.0" rpy="0 0 0" />
+        <axis xyz="0 0 1" />
+    </joint>
+    <joint name="column_back_screen_holder_3_joint" type="fixed">
+      <parent link="column_back_screen_holder_2"/>
+      <child link="column_back_screen_holder_3"/>
+        <origin xyz="-0.114 0.08 0.0" rpy="0 0.3 0" />
+        <axis xyz="0 0 1" />
+    </joint>
     <joint name="palbator_arm_hri_screen_joint" type="fixed">
       <parent link="palbator_arm_column"/>
       <child link="hri_screen_link"/>
-        <origin xyz="-0.18 0.0 0.8" rpy="1.27 0 -1.57" />
+        <origin xyz="-0.14 -0.025 0.8" rpy="1.27 0 -1.57" />
         <axis xyz="0 0 1" />
     </joint>
@@ -38,4 +148,16 @@
       </visual>
     </gazebo>
+  <gazebo reference="column_back_screen_holder_1">
+    <material>Gazebo/Black</material>
+  </gazebo>
+  <gazebo reference="column_back_screen_holder_2">
+    <material>Gazebo/Black</material>
+  </gazebo>
+  <gazebo reference="column_back_screen_holder_3">
+    <material>Gazebo/Black</material>
+  </gazebo>
+  <gazebo reference="column_back_screen_holder_4">
+    <material>Gazebo/Black</material>
+  </gazebo>
   </xacro:macro>
 </robot>

Commit message: added new urdf and fix

File: pmb2_robot/pmb2_description/urdf/display/hri_screen.urdf.xacro (robot description, xacro)
@@ -94,5 +94,5 @@
         <origin xyz="0 0 0" rpy="0 0 0" />
         <geometry>
-            <box size="0.02 -0.14 0.04"/>
+            <box size="0.02 0.14 0.04"/>
         </geometry>
         <material name="black">
