Commit message: ajout gripper

File: pmb2_robot/pmb2_description/urdf/base/base.urdf.xacro (robot description, xacro)
@@ -9,5 +9,6 @@
 <robot xmlns:xacro="http://ros.org/wiki/xacro">
   <!-- Palbator arm -->
-  <xacro:include filename="$(find pmb2_description)/urdf/arm/palbator_arm.urdf.xacro"/>
+  <xacro:include filename="$(find pmb2_description)/urdf/arm/palbator_arm_with_gripper.urdf.xacro"/>
+  <!-- <xacro:include filename="$(find pmb2_description)/urdf/arm/palbator_arm.urdf.xacro"/>-->
   <xacro:include filename="$(find pmb2_description)/urdf/deg_to_rad.xacro"/>
   <xacro:include filename="$(find pmb2_description)/urdf/wheels/wheel.urdf.xacro"/>

File: pmb2_robot/pmb2_description/urdf/gripper/gripper.urdf.xacro (robot description, xacro)
@@ -26,5 +26,5 @@
       </visual>
       <collision>
-        <origin xyz="0 0 0" rpy="0 0 0" />
+        <origin xyz="0 0.0275 0.012" rpy="0 0 0" />
         <geometry>
           <mesh filename="package://pmb2_description/meshes/gripper/gripper_base_link.STL" />
@@ -82,5 +82,5 @@
       </visual>
       <collision>
-        <origin xyz="0 0 0" rpy="0 0 0" />
+        <origin xyz="-0.013 0.03 0.022" rpy="1.5707 1.5707 0" />
         <geometry>
           <mesh filename="package://pmb2_description/meshes/gripper/hand1_link.STL" />
@@ -110,5 +110,5 @@
       </visual>
       <collision>
-        <origin xyz="0 0 0" rpy="0 0 0" />
+        <origin xyz="0 0 0" rpy="1.5708 0 3.141592" />
         <geometry>
           <mesh filename="package://pmb2_description/meshes/gripper/fingertip1_1_link.STL" />
@@ -138,5 +138,5 @@
       </visual>
       <collision>
-        <origin xyz="0 0 0" rpy="0 0 0" />
+        <origin xyz="0 0 0" rpy="-1.5708 0 3.141592" />
         <geometry>
           <mesh filename="package://pmb2_description/meshes/gripper/fingertip1_2_link.STL" />
@@ -194,5 +194,5 @@
       </visual>
       <collision>
-        <origin xyz="0 0 0" rpy="0 0 0" />
+        <origin xyz="-0.013 0.03 0.022" rpy="1.5707 1.5707 0" />
         <geometry>
           <mesh filename="package://pmb2_description/meshes/gripper/hand2_link.STL" />
@@ -222,5 +222,5 @@
       </visual>
       <collision>
-        <origin xyz="0 0 0" rpy="0 0 0" />
+        <origin xyz="0 0 0" rpy="1.5708 0 3.141592" />
         <geometry>
           <mesh filename="package://pmb2_description/meshes/gripper/fingertip2_1_link.STL" />
@@ -251,5 +251,5 @@
       </visual>
       <collision>
-        <origin xyz="0 0 0" rpy="0 0 0" />
+        <origin xyz="0 0 0" rpy="-1.5708 0 3.141592" />
         <geometry>
           <mesh filename="package://pmb2_description/meshes/gripper/fingertip2_2_link.STL" />
@@ -271,10 +271,10 @@
       <axis xyz="0 0 0" />
     </joint>
-    <joint name="motor1_hand_joint" type="fixed">
+    <joint name="motor1_hand_joint" type="revolute">
       <origin xyz="0 0 0" rpy="0 0 0" />
       <parent link="motor1_link" />
       <child link="hand1_link" />
       <axis xyz="0 0 1" />
-      <!-- <limit lower="-1" upper="1" effort="10" velocity="0.5" /> -->
+      <limit lower="-1" upper="1" effort="10" velocity="0.5" />
     </joint>
     <joint name="hand1_fingertip1_joint" type="fixed">
@@ -283,5 +283,5 @@
       <child link="fingertip1_1_link" />
       <axis xyz="0 0 1" />
-      <!-- <limit lower="-1" upper="1" effort="10" velocity="0.5" /> -->
+      <!--<limit lower="-1" upper="1" effort="10" velocity="0.5" />-->
     </joint>
     <joint name="hand1_fingertip2_joint" type="fixed">
@@ -290,5 +290,5 @@
       <child link="fingertip1_2_link" />
       <axis xyz="0 0 1" />
-      <!-- <limit lower="-1" upper="1" effort="10" velocity="0.5" /> -->
+      <!--<limit lower="-1" upper="1" effort="10" velocity="0.5" />-->
     </joint>
     <joint name="gripper_motor2_joint" type="fixed">
@@ -298,10 +298,10 @@
       <axis xyz="0 0 0" />
     </joint>
-    <joint name="motor2_hand_joint" type="fixed">
+    <joint name="motor2_hand_joint" type="revolute">
       <origin xyz="0 0 0" rpy="0 0 0" />
       <parent link="motor2_link" />
       <child  link="hand2_link" />
       <axis xyz="0 0 1" />
-      <!-- <limit lower="-1" upper="1" effort="10" velocity="0.5" /> -->
+      <limit lower="-1" upper="1" effort="10" velocity="0.5" />
     </joint>
     <joint name="hand2_fingertip1_joint" type="fixed">
@@ -310,5 +310,5 @@
       <child link="fingertip2_1_link" />
       <axis xyz="0 0 1" />
-      <!-- <limit lower="-1" upper="1" effort="10" velocity="0.5" /> -->
+      <!--<limit lower="-1" upper="1" effort="10" velocity="0.5" />-->
     </joint>
     <joint name="hand2_fingertip2_joint" type="fixed">
@@ -317,5 +317,5 @@
       <child link="fingertip2_2_link" />
       <axis xyz="0 0 1" />
-      <!-- <limit lower="-1" upper="1" effort="10" velocity="0.5" /> -->
+      <!--<limit lower="-1" upper="1" effort="10" velocity="0.5" />-->
     </joint>
     <!-- TRANSMISSIONS -->
@@ -331,5 +331,5 @@
     </transmission>
     <!-- TRANSMISSIONS FOR LEFT AND RIGHT FINGERS MAIN MOTORS-->
-    <!-- <transmission name="left_finger_transmission">
+    <transmission name="left_finger_transmission">
       <type>SimpleTransmission</type>
       <joint name="motor1_hand_joint">
@@ -350,7 +350,8 @@
         <mechanicalReduction>1</mechanicalReduction>
       </actuator>
-    </transmission> -->
+    </transmission>
     <!-- TRANSMISSIONS FOR FINGERTIPS-->
-    <!-- <transmission name="right_finger_fingertip1_transmission">
+  <!--
+  <transmission name="right_finger_fingertip1_transmission">
       <type>SimpleTransmission</type>
       <joint name="hand2_fingertip1_joint">
@@ -391,5 +392,6 @@
         <mechanicalReduction>1</mechanicalReduction>
       </actuator>
-    </transmission> -->
+    </transmission>
+  -->
     <!-- GAZEBO MATERIAL PARAMS -->
     <gazebo reference="gripper_base_link">

Commit message: ajout troisième caméra sur la base

File: pmb2_robot/pmb2_description/urdf/base/base.urdf.xacro (robot description, xacro)
@@ -99,4 +99,81 @@
     <!-- Palbator arm -->
     <xacro:palbator_arm parent="${name}_link" />
+    <!-- Base Camera-->
+    <link name="palbator_base_camera_link" >
+      <inertial>
+          <origin xyz="0 0 0" rpy="0 0 0"/>
+          <mass value="0.1"/>
+          <inertia ixx="0.1" ixy="0" ixz="0" iyy="0.1" iyz="0" izz="0.1"/>
+      </inertial>
+        <visual>
+            <geometry>
+              <box size="0.03 0.18 0.02"/>
+          </geometry>
+          <material name="Black">
+            <color rgba="0 0 0 1.0"/>
+          </material>
+            <origin xyz="0 0 0" rpy="0 0 0"/>
+        </visual>
+    </link>
+     <!-- JOINTS -->
+    <joint name="palbator_base_camera_joint" type="fixed">
+      <parent link="${name}_link"/>
+      <child link="palbator_base_camera_link"/>
+      <origin xyz="0.25 0.0 0.23" rpy="0 0.35 0.0" />
+      <axis xyz="0 0 0" />
+    </joint>
+    <!-- Empty camera joint for fixing wrong depth sensor orientation -->
+    <joint name="camera_depth_joint_2" type="fixed">
+      <origin xyz="0 0 0" rpy="${-PI/2} 0 ${-PI/2} "/>
+      <parent link="palbator_base_camera_link"/>
+      <child link="camera_depth_link_2"/>
+    </joint>
+    <link name="camera_depth_link_2"></link>
+    <!-- GAZEBO MATERIALS -->
+    <gazebo reference="palbator_base_camera_link">
+      <material>Gazebo/Black</material>
+    </gazebo>
+    <!-- GAZEBO PLUGINS -->
+    <gazebo reference="palbator_base_camera_link">
+    <sensor name="palbator_base_camera_link_camera" type="depth">
+      <update_rate>20</update_rate>
+      <camera>
+        <horizontal_fov>1.047198</horizontal_fov>
+        <image>
+          <width>640</width>
+          <height>480</height>
+          <format>R8G8B8</format>
+        </image>
+        <clip>
+          <near>0.05</near>
+          <far>5.0</far>
+        </clip>
+      </camera>
+      <plugin name="camera_plugin" filename="libgazebo_ros_openni_kinect.so">
+        <baseline>0.2</baseline>
+        <alwaysOn>true</alwaysOn>
+        <updateRate>20.0</updateRate>
+        <cameraName>camera_ir_base</cameraName>
+        <imageTopicName>/camera_base/color/image_raw</imageTopicName>
+        <cameraInfoTopicName>/camera_base/color/camera_info</cameraInfoTopicName>
+        <depthImageTopicName>/camera_base/depth/image_raw</depthImageTopicName>
+        <depthImageCameraInfoTopicName>/camera_base/depth/camera_info</depthImageCameraInfoTopicName>
+        <pointCloudTopicName>/camera_base/depth/points</pointCloudTopicName>
+        <frameName>camera_depth_link_2</frameName>
+        <pointCloudCutoff>0.5</pointCloudCutoff>
+        <pointCloudCutoffMax>3.0</pointCloudCutoffMax>
+        <distortionK1>0</distortionK1>
+        <distortionK2>0</distortionK2>
+        <distortionK3>0</distortionK3>
+        <distortionT1>0</distortionT1>
+        <distortionT2>0</distortionT2>
+        <CxPrime>0</CxPrime>
+        <Cx>0</Cx>
+        <Cy>0</Cy>
+        <focalLength>0</focalLength>
+        <hackBaseline>0</hackBaseline>
+      </plugin>
+    </sensor>
+    </gazebo>
   </xacro:macro>
 </robot>

Commit message: ajout camera

File: pmb2_robot/pmb2_description/urdf/base/base.urdf.xacro (robot description, xacro)
@@ -100,4 +100,81 @@
     <!-- Palbator arm -->
     <xacro:palbator_arm parent="${name}_link" />
+    <!-- Base Camera-->
+    <link name="palbator_base_camera_link" >
+      <inertial>
+          <origin xyz="0 0 0" rpy="0 0 0"/>
+          <mass value="0.1"/>
+          <inertia ixx="0.1" ixy="0" ixz="0" iyy="0.1" iyz="0" izz="0.1"/>
+      </inertial>
+        <visual>
+            <geometry>
+              <box size="0.03 0.18 0.02"/>
+          </geometry>
+          <material name="Black">
+            <color rgba="0 0 0 1.0"/>
+          </material>
+            <origin xyz="0 0 0" rpy="0 0 0"/>
+        </visual>
+    </link>
+     <!-- JOINTS -->
+    <joint name="palbator_base_camera_joint" type="fixed">
+      <parent link="${name}_link"/>
+      <child link="palbator_base_camera_link"/>
+      <origin xyz="0.25 0.0 0.23" rpy="0 0.35 0.0" />
+      <axis xyz="0 0 0" />
+    </joint>
+    <!-- Empty camera joint for fixing wrong depth sensor orientation -->
+    <joint name="camera_depth_joint_2" type="fixed">
+      <origin xyz="0 0 0" rpy="${-PI/2} 0 ${-PI/2} "/>
+      <parent link="palbator_base_camera_link"/>
+      <child link="camera_depth_link_2"/>
+    </joint>
+    <link name="camera_depth_link_2"></link>
+    <!-- GAZEBO MATERIALS -->
+    <gazebo reference="palbator_base_camera_link">
+      <material>Gazebo/Black</material>
+    </gazebo>
+    <!-- GAZEBO PLUGINS -->
+    <gazebo reference="palbator_base_camera_link">
+    <sensor name="palbator_base_camera_link_camera" type="depth">
+      <update_rate>20</update_rate>
+      <camera>
+        <horizontal_fov>1.047198</horizontal_fov>
+        <image>
+          <width>640</width>
+          <height>480</height>
+          <format>R8G8B8</format>
+        </image>
+        <clip>
+          <near>0.05</near>
+          <far>5.0</far>
+        </clip>
+      </camera>
+      <plugin name="camera_plugin" filename="libgazebo_ros_openni_kinect.so">
+        <baseline>0.2</baseline>
+        <alwaysOn>true</alwaysOn>
+        <updateRate>20.0</updateRate>
+        <cameraName>camera_ir_base</cameraName>
+        <imageTopicName>/camera_base/color/image_raw</imageTopicName>
+        <cameraInfoTopicName>/camera_base/color/camera_info</cameraInfoTopicName>
+        <depthImageTopicName>/camera_base/depth/image_raw</depthImageTopicName>
+        <depthImageCameraInfoTopicName>/camera_base/depth/camera_info</depthImageCameraInfoTopicName>
+        <pointCloudTopicName>/camera_base/depth/points</pointCloudTopicName>
+        <frameName>camera_depth_link_2</frameName>
+        <pointCloudCutoff>0.5</pointCloudCutoff>
+        <pointCloudCutoffMax>3.0</pointCloudCutoffMax>
+        <distortionK1>0</distortionK1>
+        <distortionK2>0</distortionK2>
+        <distortionK3>0</distortionK3>
+        <distortionT1>0</distortionT1>
+        <distortionT2>0</distortionT2>
+        <CxPrime>0</CxPrime>
+        <Cx>0</Cx>
+        <Cy>0</Cy>
+        <focalLength>0</focalLength>
+        <hackBaseline>0</hackBaseline>
+      </plugin>
+    </sensor>
+    </gazebo>
   </xacro:macro>
 </robot>

Commit message: add 20kg battery pack

File: pmb2_robot/pmb2_description/urdf/base/base.urdf.xacro (robot description, xacro)
@@ -117,4 +117,21 @@
         </visual>
     </link>
+    <!-- Battery pack-->
+    <link name="palbator_base_battery_link" >
+      <inertial>
+          <origin xyz="0 0 0" rpy="0 0 0"/>
+          <mass value="20"/>
+          <inertia ixx="0.142" ixy="217" ixz="0.188" iyy="0.142" iyz="0.104" izz="0.142"/>
+      </inertial>
+        <visual>
+            <geometry>
+              <box size="0.28 0.14 0.15"/>
+          </geometry>
+          <material name="Blue">
+            <color rgba="0 0 1 1.0"/>
+          </material>
+            <origin xyz="0 0 0" rpy="0 0 0"/>
+        </visual>
+    </link>
      <!-- JOINTS -->
     <joint name="palbator_base_camera_joint" type="fixed">
@@ -122,4 +139,10 @@
       <child link="palbator_base_camera_link"/>
       <origin xyz="0.25 0.0 0.23" rpy="0 0.35 0.0" />
+      <axis xyz="0 0 0" />
+    </joint>
+      <joint name="palbator_base_battery_joint" type="fixed">
+      <parent link="${name}_link"/>
+      <child link="palbator_base_battery_link"/>
+      <origin xyz="0.0 0.0 0.025" rpy="0 0.0 0.0" />
       <axis xyz="0 0 0" />
     </joint>

Commit message: fix shaking

File: pmb2_robot/pmb2_description/urdf/base/base.urdf.xacro (robot description, xacro)
@@ -122,5 +122,5 @@
           <origin xyz="0 0 0" rpy="0 0 0"/>
           <mass value="20"/>
-          <inertia ixx="0.142" ixy="217" ixz="0.188" iyy="0.142" iyz="0.104" izz="0.142"/>
+          <inertia ixx="0.142" ixy="0.217" ixz="0.188" iyy="0.142" iyz="0.104" izz="0.142"/>
       </inertial>
         <visual>

Commit message: delete useless import, changed camera position

File: pmb2_robot/pmb2_description/urdf/base/base.urdf.xacro (robot description, xacro)
@@ -138,5 +138,5 @@
       <parent link="${name}_link"/>
       <child link="palbator_base_camera_link"/>
-      <origin xyz="0.25 0.0 0.23" rpy="0 0.35 0.0" />
+      <origin xyz="0.25 0.0 0.2" rpy="0 0.55 0.0" />
       <axis xyz="0 0 0" />
     </joint>

Commit message: update base camera parameters

File: pmb2_robot/pmb2_description/urdf/base/base.urdf.xacro (robot description, xacro)
@@ -138,5 +138,5 @@
       <parent link="${name}_link"/>
       <child link="palbator_base_camera_link"/>
-      <origin xyz="0.25 0.0 0.2" rpy="0 0.55 0.0" />
+      <origin xyz="0.245 0.0 0.215" rpy="0 0.75 0.0" />
       <axis xyz="0 0 0" />
     </joint>
@@ -163,5 +163,5 @@
       <update_rate>20</update_rate>
       <camera>
-        <horizontal_fov>1.047198</horizontal_fov>
+        <horizontal_fov>1.570797</horizontal_fov>
         <image>
           <width>640</width>
@@ -185,5 +185,5 @@
         <pointCloudTopicName>/camera_base/depth/points</pointCloudTopicName>
         <frameName>camera_depth_link_2</frameName>
-        <pointCloudCutoff>0.05</pointCloudCutoff>
+        <pointCloudCutoff>0.225</pointCloudCutoff>
         <pointCloudCutoffMax>3.0</pointCloudCutoffMax>
         <distortionK1>0</distortionK1>
