Commit message: Fix nav

File: pmb2_robot/pmb2_description/urdf/wheels/caster.gazebo.xacro (robot description, xacro)
@@ -11,22 +11,22 @@
     <!-- Contact model for the caster wheel surface -->
     <gazebo reference="caster_${side}_1_link">
-      <kp>1000000.0</kp>
-      <kd>1000.0</kd>
-      <mu1>1.0</mu1>
-      <mu2>1.0</mu2>
-      <fdir1>0 0 1</fdir1>
-      <maxVel>1.0</maxVel>
-      <minDepth>0.0</minDepth>
+      <kp>100000000.0</kp>
+      <kd>10.0</kd>
+      <mu1>0.1</mu1>
+      <mu2>0.1</mu2>
+      <!--<fdir1>1 0 0</fdir1>-->
+      <maxVel>10.0</maxVel>
+      <minDepth>0.0005</minDepth>
       <implicitSpringDamper>0</implicitSpringDamper>
       <material>Gazebo/DarkGrey</material>
     </gazebo>
     <gazebo reference="caster_${side}_2_link">
-      <kp>1000000.0</kp>
-      <kd>1000.0</kd>
-      <mu1>0.4</mu1>
-      <mu2>0.4</mu2>
-      <fdir1>1 0 0</fdir1>
-      <maxVel>1.0</maxVel>
-      <minDepth>0.00</minDepth>
+      <kp>10000000.0</kp>
+      <kd>10.0</kd>
+      <mu1>0.1</mu1>
+      <mu2>0.1</mu2>
+      <!--<fdir1>1 0 0</fdir1>-->
+      <maxVel>10.0</maxVel>
+      <minDepth>0.0005</minDepth>
       <implicitSpringDamper>0</implicitSpringDamper>
       <material>Gazebo/DarkGrey</material>

File: pmb2_robot/pmb2_description/urdf/wheels/caster.urdf.xacro (robot description, xacro)
@@ -50,5 +50,5 @@
         <origin xyz="0 0 0" rpy="0 0 0"/>
         <geometry>
-          <cylinder radius="${radius}" length="${width}"/>
+	  <sphere radius="${radius}" />
         </geometry>
       </collision>

File: pmb2_robot/pmb2_description/urdf/wheels/wheel.gazebo.xacro (robot description, xacro)
@@ -12,10 +12,10 @@
     <gazebo reference="wheel_${side}_link">
       <kp>1000000.0</kp>
-      <kd>1000.0</kd>
-      <mu1>1.0</mu1>
-      <mu2>1.0</mu2>
-      <fdir1>1 0 0</fdir1>
+      <kd>100.0</kd>
+      <mu1>100000000000000.0</mu1>
+      <mu2>100000000000000.0</mu2>
+      <!--<fdir1>1 0 0</fdir1>-->
       <maxVel>1.0</maxVel>
-      <minDepth>0.00</minDepth>
+      <minDepth>0.002</minDepth>
       <implicitSpringDamper>1</implicitSpringDamper>
       <material>Gazebo/DarkGrey</material>

File: pmb2_robot/pmb2_description/urdf/wheels/wheel.urdf.xacro (robot description, xacro)
@@ -29,5 +29,5 @@
           <origin xyz="0 0 0" rpy="0 0 0"/>
           <geometry>
-            <cylinder radius="${radius}" length="${width}"/>
+            <sphere radius="${radius}" /> <!-- length="${width}"/> -->
           </geometry>
         </collision>
@@ -60,5 +60,5 @@
           <parent link="suspension_${side}_link"/>
           <child link="wheel_${side}_link"/>
-          <origin xyz="0 ${-separation / 2 * reflect} 0" rpy="${-90.0 * deg_to_rad} 0 0"/>
+          <origin xyz="0 ${-separation / 2 * reflect} 0.0" rpy="${-90.0 * deg_to_rad} 0 0"/>
           <axis xyz="0 0 1"/>
           <limit effort="${torque}" velocity="${velocity / radius}"/>
