Commit message: Update gripper xacro

File: pmb2_robot/pmb2_description/urdf/gripper/gripper.urdf.xacro (robot description, xacro)
@@ -5,5 +5,5 @@
     <link name="gripper_base_link">
       <inertial>
-        <origin xyz="-9.6291E-09 -0.00038057 -0.015989" rpy="0 0 0" />
+        <origin xyz="0 0 0" rpy="0 0 0" />
         <mass value="0.080698" />
         <inertia
@@ -320,4 +320,14 @@
     </joint>
     <!-- TRANSMISSIONS -->
+    <transmission name="tran7">
+      <type>SimpleTransmission</type>
+      <joint name="palbator_arm_wrist_3_joint">
+        <hardwareInterface>hardware_interface/EffortJointInterface</hardwareInterface>
+      </joint>
+      <actuator name="motor7">
+        <hardwareInterface>hardware_interface/EffortJointInterface</hardwareInterface>
+        <mechanicalReduction>1</mechanicalReduction>
+      </actuator>
+    </transmission>
     <transmission name="left_finger_transmission">
       <type>SimpleTransmission</type>

Commit message: Updating controllers gazebo for Palbator gripper

File: pmb2_robot/pmb2_description/urdf/gripper/gripper.urdf.xacro (robot description, xacro)
@@ -351,4 +351,45 @@
       </actuator>
     </transmission>
+    <!-- TRANSMISSIONS FOR FINGERTIPS-->
+    <!-- <transmission name="right_finger_fingertip1_transmission">
+      <type>SimpleTransmission</type>
+      <joint name="hand2_fingertip1_joint">
+        <hardwareInterface>hardware_interface/EffortJointInterface</hardwareInterface>
+      </joint>
+      <actuator name="right_finger1">
+        <hardwareInterface>hardware_interface/EffortJointInterface</hardwareInterface>
+        <mechanicalReduction>1</mechanicalReduction>
+      </actuator>
+    </transmission>
+    <transmission name="right_finger_fingertip2_transmission">
+      <type>SimpleTransmission</type>
+      <joint name="hand2_fingertip2_joint">
+        <hardwareInterface>hardware_interface/EffortJointInterface</hardwareInterface>
+      </joint>
+      <actuator name="right_finger2">
+        <hardwareInterface>hardware_interface/EffortJointInterface</hardwareInterface>
+        <mechanicalReduction>1</mechanicalReduction>
+      </actuator>
+    </transmission>
+    <transmission name="left_finger_fingertip1_transmission">
+      <type>SimpleTransmission</type>
+      <joint name="hand1_fingertip1_joint">
+        <hardwareInterface>hardware_interface/EffortJointInterface</hardwareInterface>
+      </joint>
+      <actuator name="left_finger1">
+        <hardwareInterface>hardware_interface/EffortJointInterface</hardwareInterface>
+        <mechanicalReduction>1</mechanicalReduction>
+      </actuator>
+    </transmission>
+    <transmission name="left_finger_fingertip2_transmission">
+      <type>SimpleTransmission</type>
+      <joint name="hand1_fingertip2_joint">
+        <hardwareInterface>hardware_interface/EffortJointInterface</hardwareInterface>
+      </joint>
+      <actuator name="left_finger2">
+        <hardwareInterface>hardware_interface/EffortJointInterface</hardwareInterface>
+        <mechanicalReduction>1</mechanicalReduction>
+      </actuator>
+    </transmission> -->
     <!-- GAZEBO MATERIAL PARAMS -->
     <gazebo reference="gripper_base_link">

Commit message: Updating xacro gripper

File: pmb2_robot/pmb2_description/urdf/gripper/gripper.urdf.xacro (robot description, xacro)
@@ -271,25 +271,24 @@
       <axis xyz="0 0 0" />
     </joint>
-    <joint name="motor1_hand_joint" type="revolute">
+    <joint name="motor1_hand_joint" type="fixed">
       <origin xyz="0 0 0" rpy="0 0 0" />
       <parent link="motor1_link" />
       <child link="hand1_link" />
       <axis xyz="0 0 1" />
-      <limit lower="-1" upper="1" effort="10" velocity="0.5" />
-    </joint>
-    <joint name="hand1_fingertip1_joint" type="revolute">
+      <!-- <limit lower="-1" upper="1" effort="10" velocity="0.5" /> -->
+    </joint>
+    <joint name="hand1_fingertip1_joint" type="fixed">
       <origin xyz="-0.0056 0.0877 0.0055" rpy="0 0 0" />
       <parent link="hand1_link" />
       <child link="fingertip1_1_link" />
       <axis xyz="0 0 1" />
-      <limit lower="-1" upper="1" effort="10" velocity="0.5" />
-    </joint>
-    <joint name="hand1_fingertip2_joint"
-      type="revolute">
+      <!-- <limit lower="-1" upper="1" effort="10" velocity="0.5" /> -->
+    </joint>
+    <joint name="hand1_fingertip2_joint" type="fixed">
       <origin xyz="-0.0056 0.0877 -0.0055" rpy="0 0 0" />
       <parent link="hand1_link" />
       <child link="fingertip1_2_link" />
       <axis xyz="0 0 1" />
-      <limit lower="-1" upper="1" effort="10" velocity="0.5" />
+      <!-- <limit lower="-1" upper="1" effort="10" velocity="0.5" /> -->
     </joint>
     <joint name="gripper_motor2_joint" type="fixed">
@@ -299,24 +298,24 @@
       <axis xyz="0 0 0" />
     </joint>
-    <joint name="motor2_hand_joint" type="revolute">
+    <joint name="motor2_hand_joint" type="fixed">
       <origin xyz="0 0 0" rpy="0 0 0" />
       <parent link="motor2_link" />
       <child  link="hand2_link" />
       <axis xyz="0 0 1" />
-      <limit lower="-1" upper="1" effort="10" velocity="0.5" />
-    </joint>
-    <joint name="hand2_fingertip1_joint" type="revolute">
+      <!-- <limit lower="-1" upper="1" effort="10" velocity="0.5" /> -->
+    </joint>
+    <joint name="hand2_fingertip1_joint" type="fixed">
       <origin xyz="-0.0056 0.0877 0.0055" rpy="0 0 0" />
       <parent link="hand2_link" />
       <child link="fingertip2_1_link" />
       <axis xyz="0 0 1" />
-      <limit lower="-1" upper="1" effort="10" velocity="0.5" />
-    </joint>
-    <joint name="hand2_fingertip2_joint" type="revolute">
+      <!-- <limit lower="-1" upper="1" effort="10" velocity="0.5" /> -->
+    </joint>
+    <joint name="hand2_fingertip2_joint" type="fixed">
       <origin xyz="-0.0056 0.0877 -0.0055" rpy="0 0 0" />
       <parent link="hand2_link" />
       <child link="fingertip2_2_link" />
       <axis xyz="0 0 1" />
-      <limit lower="-1" upper="1" effort="10" velocity="0.5" />
+      <!-- <limit lower="-1" upper="1" effort="10" velocity="0.5" /> -->
     </joint>
     <!-- TRANSMISSIONS -->
@@ -331,5 +330,6 @@
       </actuator>
     </transmission>
-    <transmission name="left_finger_transmission">
+    <!-- TRANSMISSIONS FOR LEFT AND RIGHT FINGERS MAIN MOTORS-->
+    <!-- <transmission name="left_finger_transmission">
       <type>SimpleTransmission</type>
       <joint name="motor1_hand_joint">
@@ -350,5 +350,5 @@
         <mechanicalReduction>1</mechanicalReduction>
       </actuator>
-    </transmission>
+    </transmission> -->
     <!-- TRANSMISSIONS FOR FINGERTIPS-->
     <!-- <transmission name="right_finger_fingertip1_transmission">

Commit message: ajout mouvement de saisi d'objet

File: pmb2_robot/pmb2_description/urdf/gripper/gripper.urdf.xacro (robot description, xacro)
@@ -256,4 +256,6 @@
         </geometry>
       </collision>
+    </link>
+    <link name="end_effector_link">
     </link>
     <!-- JOINTS -->
@@ -319,4 +321,9 @@
       <!--<limit lower="-1" upper="1" effort="10" velocity="0.5" />-->
     </joint>
+    <joint name="gripper_end_effector_joint" type="fixed">
+      <origin xyz="0 0.10 0" rpy="0 0 1.5707" />
+      <parent link="gripper_base_link" />
+      <child link="end_effector_link" />
+    </joint>
     <!-- TRANSMISSIONS -->
     <transmission name="tran7">
@@ -396,4 +403,5 @@
     <!-- GAZEBO MATERIAL PARAMS -->
     <gazebo reference="gripper_base_link">
+      <self_collide>true</self_collide>
       <material>Gazebo/Black</material>
     </gazebo>

Commit message: fingertip libre, ajout grip

File: pmb2_robot/pmb2_description/urdf/gripper/gripper.urdf.xacro (robot description, xacro)
@@ -280,5 +280,5 @@
       <limit lower="-1" upper="1" effort="10" velocity="0.5" />
     </joint>
-    <joint name="hand1_fingertip1_joint" type="fixed">
+    <joint name="hand1_fingertip1_joint" type="revolute">
       <origin xyz="-0.0056 0.0877 0.0055" rpy="0 0 0" />
       <parent link="hand1_link" />
@@ -287,5 +287,5 @@
       <!--<limit lower="-1" upper="1" effort="10" velocity="0.5" />-->
     </joint>
-    <joint name="hand1_fingertip2_joint" type="fixed">
+    <joint name="hand1_fingertip2_joint" type="revolute">
       <origin xyz="-0.0056 0.0877 -0.0055" rpy="0 0 0" />
       <parent link="hand1_link" />
@@ -307,5 +307,5 @@
       <limit lower="-1" upper="1" effort="10" velocity="0.5" />
     </joint>
-    <joint name="hand2_fingertip1_joint" type="fixed">
+    <joint name="hand2_fingertip1_joint" type="revolute">
       <origin xyz="-0.0056 0.0877 0.0055" rpy="0 0 0" />
       <parent link="hand2_link" />
@@ -314,5 +314,5 @@
       <!--<limit lower="-1" upper="1" effort="10" velocity="0.5" />-->
     </joint>
-    <joint name="hand2_fingertip2_joint" type="fixed">
+    <joint name="hand2_fingertip2_joint" type="revolute">
       <origin xyz="-0.0056 0.0877 -0.0055" rpy="0 0 0" />
       <parent link="hand2_link" />
@@ -359,5 +359,4 @@
     </transmission>
     <!-- TRANSMISSIONS FOR FINGERTIPS-->
-  <!--
   <transmission name="right_finger_fingertip1_transmission">
       <type>SimpleTransmission</type>
@@ -400,26 +399,52 @@
       </actuator>
     </transmission>
-  -->
     <!-- GAZEBO MATERIAL PARAMS -->
     <gazebo reference="gripper_base_link">
-      <self_collide>true</self_collide>
+      <mu1>100.0</mu1>
+      <mu2>50.0</mu2>
+      <minDepth>0.003</minDepth>
+      <maxVel>2</maxVel>
       <material>Gazebo/Black</material>
     </gazebo>
     <gazebo reference="hand2_link">
+      <mu1>100.0</mu1>
+      <mu2>50.0</mu2>
+      <minDepth>0.003</minDepth>
+      <maxVel>2</maxVel>
       <material>Gazebo/LightBlue</material>
     </gazebo>
     <gazebo reference="hand1_link">
+      <mu1>100.0</mu1>
+      <mu2>50.0</mu2>
+      <minDepth>0.003</minDepth>
+      <maxVel>2</maxVel>
       <material>Gazebo/LightBlue</material>
     </gazebo>
     <gazebo reference="fingertip1_1_link">
+      <mu1>100.0</mu1>
+      <mu2>50.0</mu2>
+      <minDepth>0.003</minDepth>
+      <maxVel>2</maxVel>
       <material>Gazebo/Grey</material>
     </gazebo>
     <gazebo reference="fingertip1_2_link">
+      <mu1>100.0</mu1>
+      <mu2>50.0</mu2>
+      <minDepth>0.003</minDepth>
+      <maxVel>2</maxVel>
       <material>Gazebo/Grey</material>
     </gazebo>
     <gazebo reference="fingertip2_1_link">
+      <mu1>100.0</mu1>
+      <mu2>50.0</mu2>
+      <minDepth>0.003</minDepth>
+      <maxVel>2</maxVel>
       <material>Gazebo/Grey</material>
     </gazebo>
     <gazebo reference="fingertip2_2_link">
+      <mu1>100.0</mu1>
+      <mu2>50.0</mu2>
+      <minDepth>0.003</minDepth>
+      <maxVel>2</maxVel>
       <material>Gazebo/Grey</material>
     </gazebo>

Commit message: update

File: pmb2_robot/pmb2_description/urdf/gripper/gripper.urdf.xacro (robot description, xacro)
@@ -285,5 +285,5 @@
       <child link="fingertip1_1_link" />
       <axis xyz="0 0 1" />
-      <!--<limit lower="-1" upper="1" effort="10" velocity="0.5" />-->
+      <limit lower="-1" upper="1" effort="10" velocity="0.5" />
     </joint>
     <joint name="hand1_fingertip2_joint" type="revolute">
@@ -292,5 +292,5 @@
       <child link="fingertip1_2_link" />
       <axis xyz="0 0 1" />
-      <!--<limit lower="-1" upper="1" effort="10" velocity="0.5" />-->
+      <limit lower="-1" upper="1" effort="10" velocity="0.5" />
     </joint>
     <joint name="gripper_motor2_joint" type="fixed">
@@ -312,5 +312,5 @@
       <child link="fingertip2_1_link" />
       <axis xyz="0 0 1" />
-      <!--<limit lower="-1" upper="1" effort="10" velocity="0.5" />-->
+      <limit lower="-1" upper="1" effort="10" velocity="0.5" />
     </joint>
     <joint name="hand2_fingertip2_joint" type="revolute">
@@ -319,5 +319,5 @@
       <child link="fingertip2_2_link" />
       <axis xyz="0 0 1" />
-      <!--<limit lower="-1" upper="1" effort="10" velocity="0.5" />-->
+      <limit lower="-1" upper="1" effort="10" velocity="0.5" />
     </joint>
     <joint name="gripper_end_effector_joint" type="fixed">
@@ -401,51 +401,47 @@
     <!-- GAZEBO MATERIAL PARAMS -->
     <gazebo reference="gripper_base_link">
+      <material>Gazebo/Black</material>
+    </gazebo>
+    <gazebo reference="hand2_link">
+      <material>Gazebo/LightBlue</m
+      <mu1>100.0</mu1>
+      <mu2>50.0</mu2>
+      <minDepth>0.003</minDepth>
+      <maxVel>2</maxVel>aterial>
+    </gazebo>
+    <gazebo reference="hand1_link">
+      <material>Gazebo/LightBlue</m
+      <mu1>100.0</mu1>
+      <mu2>50.0</mu2>
+      <minDepth>0.003</minDepth>
+      <maxVel>2</maxVel>aterial>
+    </gazebo>
+    <gazebo reference="fingertip1_1_link">
+      <material>Gazebo/Grey</material>
       <mu1>100.0</mu1>
       <mu2>50.0</mu2>
       <minDepth>0.003</minDepth>
       <maxVel>2</maxVel>
-      <material>Gazebo/Black</material>
-    </gazebo>
-    <gazebo reference="hand2_link">
+    </gazebo>
+    <gazebo reference="fingertip1_2_link">
+      <material>Gazebo/Grey</material>
       <mu1>100.0</mu1>
       <mu2>50.0</mu2>
       <minDepth>0.003</minDepth>
       <maxVel>2</maxVel>
-      <material>Gazebo/LightBlue</material>
-    </gazebo>
-    <gazebo reference="hand1_link">
+    </gazebo>
+    <gazebo reference="fingertip2_1_link">
+      <material>Gazebo/Grey</material>
       <mu1>100.0</mu1>
       <mu2>50.0</mu2>
       <minDepth>0.003</minDepth>
       <maxVel>2</maxVel>
-      <material>Gazebo/LightBlue</material>
-    </gazebo>
-    <gazebo reference="fingertip1_1_link">
+    </gazebo>
+    <gazebo reference="fingertip2_2_link">
+      <material>Gazebo/Grey</material>
       <mu1>100.0</mu1>
       <mu2>50.0</mu2>
       <minDepth>0.003</minDepth>
       <maxVel>2</maxVel>
-      <material>Gazebo/Grey</material>
-    </gazebo>
-    <gazebo reference="fingertip1_2_link">
-      <mu1>100.0</mu1>
-      <mu2>50.0</mu2>
-      <minDepth>0.003</minDepth>
-      <maxVel>2</maxVel>
-      <material>Gazebo/Grey</material>
-    </gazebo>
-    <gazebo reference="fingertip2_1_link">
-      <mu1>100.0</mu1>
-      <mu2>50.0</mu2>
-      <minDepth>0.003</minDepth>
-      <maxVel>2</maxVel>
-      <material>Gazebo/Grey</material>
-    </gazebo>
-    <gazebo reference="fingertip2_2_link">
-      <mu1>100.0</mu1>
-      <mu2>50.0</mu2>
-      <minDepth>0.003</minDepth>
-      <maxVel>2</maxVel>
-      <material>Gazebo/Grey</material>
     </gazebo>
     </xacro:macro>

Commit message: fix

File: pmb2_robot/pmb2_description/urdf/gripper/gripper.urdf.xacro (robot description, xacro)
@@ -404,16 +404,16 @@
     </gazebo>
     <gazebo reference="hand2_link">
-      <material>Gazebo/LightBlue</m
-      <mu1>100.0</mu1>
-      <mu2>50.0</mu2>
-      <minDepth>0.003</minDepth>
-      <maxVel>2</maxVel>aterial>
+      <material>Gazebo/LightBlue</material>
+      <mu1>100.0</mu1>
+      <mu2>50.0</mu2>
+      <minDepth>0.003</minDepth>
+      <maxVel>2</maxVel>
     </gazebo>
     <gazebo reference="hand1_link">
-      <material>Gazebo/LightBlue</m
-      <mu1>100.0</mu1>
-      <mu2>50.0</mu2>
-      <minDepth>0.003</minDepth>
-      <maxVel>2</maxVel>aterial>
+      <material>Gazebo/LightBlue</material>
+      <mu1>100.0</mu1>
+      <mu2>50.0</mu2>
+      <minDepth>0.003</minDepth>
+      <maxVel>2</maxVel>
     </gazebo>
     <gazebo reference="fingertip1_1_link">

Commit message: amelioration grip, ajout fingertip

File: pmb2_robot/pmb2_description/urdf/gripper/gripper.urdf.xacro (robot description, xacro)
@@ -91,12 +91,12 @@
       <inertial>
         <origin xyz="-0.0010321 0.0050002 -3.5129E-05" rpy="0 0 0" />
-        <mass value="0.0062622" />
-        <inertia
-          ixx="9.7768E-07"
-          ixy="1.568E-11"
-          ixz="1.5157E-09"
-          iyy="1.0446E-06"
-          iyz="5.6166E-12"
-          izz="1.8516E-07" />
+        <mass value="0.034799" />
+        <inertia
+          ixx="1.1668E-05"
+          ixy="1.0081E-14"
+          ixz="1.9718E-14"
+          iyy="1.5945E-05"
+          iyz="1.2429E-07"
+          izz="6.7071E-06" />
       </inertial>
       <visual>
@@ -119,12 +119,12 @@
       <inertial>
         <origin xyz="-0.0010321 0.0050002 -3.5129E-05" rpy="0 0 0" />
-        <mass value="0.0062622" />
-        <inertia
-          ixx="9.7768E-07"
-          ixy="1.5681E-11"
-          ixz="1.5157E-09"
-          iyy="1.0446E-06"
-          iyz="5.6167E-12"
-          izz="1.8516E-07" />
+        <mass value="0.034799" />
+        <inertia
+          ixx="1.1668E-05"
+          ixy="1.0081E-14"
+          ixz="1.9718E-14"
+          iyy="1.5945E-05"
+          iyz="1.2429E-07"
+          izz="6.7071E-06" />
       </inertial>
       <visual>
@@ -203,12 +203,12 @@
       <inertial>
         <origin xyz="-0.0010321375 0.0050002 -3.512856E-05" rpy="0 0 0" />
-        <mass value="0.00626220315523217" />
-        <inertia
-          ixx="9.7767596887376E-07"
-          ixy="1.56803668594996E-11"
-          ixz="1.5157444715102E-09"
-          iyy="1.04455526714601E-06"
-          iyz="5.61662128246886E-12"
-          izz="1.8516351841874E-07" />
+        <mass value="0.034799" />
+        <inertia
+          ixx="1.1668E-05"
+          ixy="1.0081E-14"
+          ixz="1.9718E-14"
+          iyy="1.5945E-05"
+          iyz="1.2429E-07"
+          izz="6.7071E-06" />
       </inertial>
       <visual>
@@ -232,12 +232,12 @@
         <origin
           xyz="-0.001032137588 0.0050002404 -3.512856642E-05" rpy="0 0 0" />
-        <mass value="0.00626220316616597" />
-        <inertia
-          ixx="9.77675969200664E-07"
-          ixy="1.56806262615851E-11"
-          ixz="1.51574413550611E-09"
-          iyy="1.04455526789645E-06"
-          iyz="5.6167744165921E-12"
-          izz="1.85163518907813E-07" />
+        <mass value="0.034799" />
+        <inertia
+          ixx="1.1668E-05"
+          ixy="1.0081E-14"
+          ixz="1.9718E-14"
+          iyy="1.5945E-05"
+          iyz="1.2429E-07"
+          izz="6.7071E-06" />
       </inertial>
       <visual>
@@ -278,5 +278,5 @@
       <child link="hand1_link" />
       <axis xyz="0 0 1" />
-      <limit lower="-1" upper="1" effort="10" velocity="0.5" />
+      <limit lower="-1" upper="1" effort="50" velocity="0.5" />
     </joint>
     <joint name="hand1_fingertip1_joint" type="revolute">
@@ -285,5 +285,5 @@
       <child link="fingertip1_1_link" />
       <axis xyz="0 0 1" />
-      <limit lower="-1" upper="1" effort="10" velocity="0.5" />
+      <limit lower="-1" upper="1" effort="0.05" velocity="0.5" />
     </joint>
     <joint name="hand1_fingertip2_joint" type="revolute">
@@ -292,5 +292,5 @@
       <child link="fingertip1_2_link" />
       <axis xyz="0 0 1" />
-      <limit lower="-1" upper="1" effort="10" velocity="0.5" />
+      <limit lower="-1" upper="1" effort="0.05" velocity="0.5" />
     </joint>
     <joint name="gripper_motor2_joint" type="fixed">
@@ -305,5 +305,5 @@
       <child  link="hand2_link" />
       <axis xyz="0 0 1" />
-      <limit lower="-1" upper="1" effort="10" velocity="0.5" />
+      <limit lower="-1" upper="1" effort="50" velocity="0.5" />
     </joint>
     <joint name="hand2_fingertip1_joint" type="revolute">
@@ -312,5 +312,5 @@
       <child link="fingertip2_1_link" />
       <axis xyz="0 0 1" />
-      <limit lower="-1" upper="1" effort="10" velocity="0.5" />
+      <limit lower="-1" upper="1" effort="0.05" velocity="0.5" />
     </joint>
     <joint name="hand2_fingertip2_joint" type="revolute">
@@ -319,5 +319,5 @@
       <child link="fingertip2_2_link" />
       <axis xyz="0 0 1" />
-      <limit lower="-1" upper="1" effort="10" velocity="0.5" />
+      <limit lower="-1" upper="1" effort="0.05" velocity="0.5" />
     </joint>
     <joint name="gripper_end_effector_joint" type="fixed">
@@ -405,43 +405,67 @@
     <gazebo reference="hand2_link">
       <material>Gazebo/LightBlue</material>
-      <mu1>100.0</mu1>
-      <mu2>50.0</mu2>
-      <minDepth>0.003</minDepth>
-      <maxVel>2</maxVel>
+      <kp>1000000</kp>
+      <kd>100</kd>
+      <mu1>100.0</mu1>
+      <mu2>50.0</mu2>
+      <slip1>1</slip1>
+      <fdir1>0 0 1</fdir1>
+      <min_depth>0.00</min_depth>
+      <max_vel>2</max_vel>
     </gazebo>
     <gazebo reference="hand1_link">
       <material>Gazebo/LightBlue</material>
-      <mu1>100.0</mu1>
-      <mu2>50.0</mu2>
-      <minDepth>0.003</minDepth>
-      <maxVel>2</maxVel>
+      <kp>1000000</kp>
+      <kd>100</kd>
+      <mu1>100.0</mu1>
+      <mu2>50.0</mu2>
+      <slip1>1</slip1>
+      <fdir1>0 0 1</fdir1>
+      <min_depth>0.00</min_depth>
+      <max_vel>2</max_vel>
     </gazebo>
     <gazebo reference="fingertip1_1_link">
       <material>Gazebo/Grey</material>
-      <mu1>100.0</mu1>
-      <mu2>50.0</mu2>
-      <minDepth>0.003</minDepth>
-      <maxVel>2</maxVel>
+      <kp>1000000</kp>
+      <kd>100</kd>
+      <mu1>100.0</mu1>
+      <mu2>50.0</mu2>
+      <slip1>1</slip1>
+      <fdir1>0 0 1</fdir1>
+      <min_depth>0.00</min_depth>
+      <max_vel>2</max_vel>
     </gazebo>
     <gazebo reference="fingertip1_2_link">
       <material>Gazebo/Grey</material>
-      <mu1>100.0</mu1>
-      <mu2>50.0</mu2>
-      <minDepth>0.003</minDepth>
-      <maxVel>2</maxVel>
+      <kp>1000000</kp>
+      <kd>100</kd>
+      <mu1>100.0</mu1>
+      <mu2>50.0</mu2>
+      <slip1>1</slip1>
+      <fdir1>0 0 1</fdir1>
+      <min_depth>0.00</min_depth>
+      <max_vel>2</max_vel>
     </gazebo>
     <gazebo reference="fingertip2_1_link">
       <material>Gazebo/Grey</material>
-      <mu1>100.0</mu1>
-      <mu2>50.0</mu2>
-      <minDepth>0.003</minDepth>
-      <maxVel>2</maxVel>
+      <kp>1000000</kp>
+      <kd>100</kd>
+      <mu1>100.0</mu1>
+      <mu2>50.0</mu2>
+      <slip1>1</slip1>
+      <fdir1>0 0 1</fdir1>
+      <min_depth>0.00</min_depth>
+      <max_vel>2</max_vel>
     </gazebo>
     <gazebo reference="fingertip2_2_link">
       <material>Gazebo/Grey</material>
-      <mu1>100.0</mu1>
-      <mu2>50.0</mu2>
-      <minDepth>0.003</minDepth>
-      <maxVel>2</maxVel>
+      <kp>1000000</kp>
+      <kd>100</kd>
+      <mu1>100.0</mu1>
+      <mu2>50.0</mu2>
+      <slip1>1</slip1>
+      <fdir1>0 0 1</fdir1>
+      <min_depth>0.00</min_depth>
+      <max_vel>2</max_vel>
     </gazebo>
     </xacro:macro>
