Commit message: change fingertip mass

File: pmb2_robot/pmb2_description/urdf/gripper/gripper.urdf.xacro (robot description, xacro)
@@ -91,5 +91,5 @@
       <inertial>
         <origin xyz="-0.0010321 0.0050002 -3.5129E-05" rpy="0 0 0" />
-        <mass value="0.034799" />
+        <mass value="0.0062622" />
         <inertia
           ixx="1.1668E-05"
@@ -119,5 +119,5 @@
       <inertial>
         <origin xyz="-0.0010321 0.0050002 -3.5129E-05" rpy="0 0 0" />
-        <mass value="0.034799" />
+        <mass value="0.0062622" />
         <inertia
           ixx="1.1668E-05"
@@ -203,5 +203,5 @@
       <inertial>
         <origin xyz="-0.0010321375 0.0050002 -3.512856E-05" rpy="0 0 0" />
-        <mass value="0.034799" />
+        <mass value="0.0062622" />
         <inertia
           ixx="1.1668E-05"
@@ -232,5 +232,5 @@
         <origin
           xyz="-0.001032137588 0.0050002404 -3.512856642E-05" rpy="0 0 0" />
-        <mass value="0.034799" />
+        <mass value="0.0062622" />
         <inertia
           ixx="1.1668E-05"

Commit message: fix arm, update gripper and wheels

File: pmb2_robot/pmb2_description/urdf/gripper/gripper.urdf.xacro (robot description, xacro)
@@ -407,54 +407,59 @@
       <self_collide>true</self_collide>
       <kp>1000000.0</kp>
-      <kd>1000.0</kd>
-      <mu1>1.0</mu1>
-      <mu2>1.0</mu2>
-      <fdir1>1 0 0</fdir1>
-      <maxVel>1.0</maxVel>
+      <kd>100.0</kd>
+      <mu1>100.0</mu1>
+      <mu2>100.0</mu2>
+      <maxVel>1.0</maxVel>
+      <minDepth>0.002</minDepth>
     </gazebo>
     <gazebo reference="hand1_link">
       <material>Gazebo/LightBlue</material>
       <self_collide>true</self_collide>
-      <kp>1000000</kp>
-      <kd>100</kd>
-      <mu1>100.0</mu1>
-      <mu2>50.0</mu2>
-      <fdir1>0 0 1</fdir1>
+      <kp>1000000.0</kp>
+      <kd>1.0</kd>
+      <mu1>100.0</mu1>
+      <mu2>100.0</mu2>
+      <maxVel>1.0</maxVel>
+      <minDepth>0.002</minDepth>
     </gazebo>
     <gazebo reference="fingertip1_1_link">
       <material>Gazebo/Grey</material>
       <self_collide>true</self_collide>
-      <kp>1000000</kp>
-      <kd>100</kd>
-      <mu1>100.0</mu1>
-      <mu2>50.0</mu2>
-      <fdir1>0 0 1</fdir1>
+      <kp>1000000.0</kp>
+      <kd>1.0</kd>
+      <mu1>100.0</mu1>
+      <mu2>100.0</mu2>
+      <maxVel>1.0</maxVel>
+      <minDepth>0.002</minDepth>
     </gazebo>
     <gazebo reference="fingertip1_2_link">
       <material>Gazebo/Grey</material>
       <self_collide>true</self_collide>
-      <kp>1000000</kp>
-      <kd>100</kd>
-      <mu1>100.0</mu1>
-      <mu2>50.0</mu2>
-      <fdir1>0 0 1</fdir1>
+      <kp>1000000.0</kp>
+      <kd>1.0</kd>
+      <mu1>100.0</mu1>
+      <mu2>100.0</mu2>
+      <maxVel>1.0</maxVel>
+      <minDepth>0.002</minDepth>
     </gazebo>
     <gazebo reference="fingertip2_1_link">
       <material>Gazebo/Grey</material>
       <self_collide>true</self_collide>
-      <kp>1000000</kp>
-      <kd>100</kd>
-      <mu1>100.0</mu1>
-      <mu2>50.0</mu2>
-      <fdir1>0 0 1</fdir1>
+      <kp>1000000.0</kp>
+      <kd>1.0</kd>
+      <mu1>100.0</mu1>
+      <mu2>100.0</mu2>
+      <maxVel>1.0</maxVel>
+      <minDepth>0.002</minDepth>
     </gazebo>
     <gazebo reference="fingertip2_2_link">
       <material>Gazebo/Grey</material>
       <self_collide>true</self_collide>
-      <kp>1000000</kp>
-      <kd>100</kd>
-      <mu1>100.0</mu1>
-      <mu2>50.0</mu2>
-      <fdir1>0 0 1</fdir1>
+      <kp>1000000.0</kp>
+      <kd>1.0</kd>
+      <mu1>100.0</mu1>
+      <mu2>100.0</mu2>
+      <maxVel>1.0</maxVel>
+      <minDepth>0.002</minDepth>
     </gazebo>
     </xacro:macro>

File: pmb2_robot/pmb2_description/urdf/wheels/caster.gazebo.xacro (robot description, xacro)
@@ -18,5 +18,4 @@
       <maxVel>10.0</maxVel>
       <minDepth>0.0005</minDepth>
-      <implicitSpringDamper>0</implicitSpringDamper>
       <material>Gazebo/DarkGrey</material>
     </gazebo>
@@ -29,6 +28,11 @@
       <maxVel>10.0</maxVel>
       <minDepth>0.0005</minDepth>
+      <material>Gazebo/DarkGrey</material>
+    </gazebo>
+    <gazebo reference="caster_{side}_1_joint">
       <implicitSpringDamper>0</implicitSpringDamper>
-      <material>Gazebo/DarkGrey</material>
+    </gazebo>
+    <gazebo reference="caster_{side}_2_joint">
+      <implicitSpringDamper>0</implicitSpringDamper>
     </gazebo>
   </xacro:macro>

File: pmb2_robot/pmb2_description/urdf/wheels/wheel.gazebo.xacro (robot description, xacro)
@@ -13,11 +13,13 @@
       <kp>1000000.0</kp>
       <kd>100.0</kd>
-      <mu1>100000000000000.0</mu1>
-      <mu2>100000000000000.0</mu2>
+      <mu1>100.0</mu1>
+      <mu2>100.0</mu2>
       <!--<fdir1>1 0 0</fdir1>-->
       <maxVel>1.0</maxVel>
       <minDepth>0.002</minDepth>
+      <material>Gazebo/DarkGrey</material>
+    </gazebo>
+    <gazebo reference="wheel_{side}_joint">
       <implicitSpringDamper>1</implicitSpringDamper>
-      <material>Gazebo/DarkGrey</material>
     </gazebo>
   </xacro:macro>

Commit message: new gripper fingertips

File: pmb2_robot/pmb2_description/urdf/gripper/gripper.urdf.xacro (robot description, xacro)
@@ -101,5 +101,5 @@
       </inertial>
       <visual>
-        <origin xyz="0 0 0" rpy="1.5708 0 3.141592" />
+        <origin xyz="0 0 0" rpy="-1.5708 0 3.141592" />
         <geometry>
           <mesh filename="package://pmb2_description/meshes/gripper/fingertip1_1_link.STL" />
@@ -110,5 +110,5 @@
       </visual>
       <collision>
-        <origin xyz="0 0 0" rpy="1.5708 0 3.141592" />
+        <origin xyz="0 0 0" rpy="-1.5708 0 3.141592" />
         <geometry>
           <mesh filename="package://pmb2_description/meshes/gripper/fingertip1_1_link.STL" />
@@ -213,5 +213,5 @@
       </inertial>
       <visual>
-        <origin xyz="0 0 0" rpy="1.5708 0 3.141592" />
+        <origin xyz="0 0 0" rpy="-1.5708 0 3.141592" />
         <geometry>
           <mesh filename="package://pmb2_description/meshes/gripper/fingertip2_1_link.STL" />
@@ -222,5 +222,5 @@
       </visual>
       <collision>
-        <origin xyz="0 0 0" rpy="1.5708 0 3.141592" />
+        <origin xyz="0 0 0" rpy="-1.5708 0 3.141592" />
         <geometry>
           <mesh filename="package://pmb2_description/meshes/gripper/fingertip2_1_link.STL" />
@@ -281,5 +281,5 @@
     </joint>
     <joint name="hand1_fingertip1_joint" type="revolute">
-      <origin xyz="-0.0056 0.0877 0.0055" rpy="0 0 0" />
+      <origin xyz="-0.0056 0.0877 0.016" rpy="0 0 0" />
       <parent link="hand1_link" />
       <child link="fingertip1_1_link" />
@@ -288,5 +288,5 @@
     </joint>
     <joint name="hand1_fingertip2_joint" type="revolute">
-      <origin xyz="-0.0056 0.0877 -0.0055" rpy="0 0 0" />
+      <origin xyz="-0.0056 0.0877 -0.006" rpy="0 0 0" />
       <parent link="hand1_link" />
       <child link="fingertip1_2_link" />
@@ -308,5 +308,5 @@
     </joint>
     <joint name="hand2_fingertip1_joint" type="revolute">
-      <origin xyz="-0.0056 0.0877 0.0055" rpy="0 0 0" />
+      <origin xyz="-0.0056 0.0877 0.016" rpy="0 0 0" />
       <parent link="hand2_link" />
       <child link="fingertip2_1_link" />
@@ -315,5 +315,5 @@
     </joint>
     <joint name="hand2_fingertip2_joint" type="revolute">
-      <origin xyz="-0.0056 0.0877 -0.0055" rpy="0 0 0" />
+      <origin xyz="-0.0056 0.0877 -0.006" rpy="0 0 0" />
       <parent link="hand2_link" />
       <child link="fingertip2_2_link" />

Commit message: tune fingertips angle limit

File: pmb2_robot/pmb2_description/urdf/gripper/gripper.urdf.xacro (robot description, xacro)
@@ -285,5 +285,5 @@
       <child link="fingertip1_1_link" />
       <axis xyz="0 0 1" />
-      <limit lower="-1" upper="1" effort="0.05" velocity="0.5" />
+      <limit lower="0" upper="0.62" effort="0.05" velocity="0.5" />
     </joint>
     <joint name="hand1_fingertip2_joint" type="revolute">
@@ -292,5 +292,5 @@
       <child link="fingertip1_2_link" />
       <axis xyz="0 0 1" />
-      <limit lower="-1" upper="1" effort="0.05" velocity="0.5" />
+      <limit lower="0" upper="0.62" effort="0.05" velocity="0.5" />
     </joint>
     <joint name="gripper_motor2_joint" type="fixed">
@@ -312,5 +312,5 @@
       <child link="fingertip2_1_link" />
       <axis xyz="0 0 1" />
-      <limit lower="-1" upper="1" effort="0.05" velocity="0.5" />
+      <limit lower="0" upper="0.62" effort="0.05" velocity="0.5" />
     </joint>
     <joint name="hand2_fingertip2_joint" type="revolute">
@@ -319,5 +319,5 @@
       <child link="fingertip2_2_link" />
       <axis xyz="0 0 1" />
-      <limit lower="-1" upper="1" effort="0.05" velocity="0.5" />
+      <limit lower="0" upper="0.62" effort="0.05" velocity="0.5" />
     </joint>
     <joint name="gripper_end_effector_joint" type="fixed">

Commit message: update grasp

File: pmb2_robot/pmb2_description/urdf/gripper/gripper.urdf.xacro (robot description, xacro)
@@ -278,5 +278,5 @@
       <child link="hand1_link" />
       <axis xyz="0 0 1" />
-      <limit lower="-1" upper="1" effort="50" velocity="0.5" />
+      <limit lower="-1" upper="1" effort="3" velocity="0.5" />
     </joint>
     <joint name="hand1_fingertip1_joint" type="revolute">
@@ -305,5 +305,5 @@
       <child  link="hand2_link" />
       <axis xyz="0 0 1" />
-      <limit lower="-1" upper="1" effort="50" velocity="0.5" />
+      <limit lower="-1" upper="1" effort="3" velocity="0.5" />
     </joint>
     <joint name="hand2_fingertip1_joint" type="revolute">
@@ -402,64 +402,43 @@
     <gazebo reference="gripper_base_link">
       <material>Gazebo/Black</material>
+      <self_collide>true</self_collide>
+      <mu1>0.9</mu1>
+      <mu2>0.9</mu2>
     </gazebo>
     <gazebo reference="hand2_link">
       <material>Gazebo/LightBlue</material>
       <self_collide>true</self_collide>
-      <kp>1000000.0</kp>
-      <kd>100.0</kd>
-      <mu1>100.0</mu1>
-      <mu2>100.0</mu2>
-      <maxVel>1.0</maxVel>
-      <minDepth>0.002</minDepth>
+      <mu1>0.9</mu1>
+      <mu2>0.9</mu2>
     </gazebo>
     <gazebo reference="hand1_link">
       <material>Gazebo/LightBlue</material>
       <self_collide>true</self_collide>
-      <kp>1000000.0</kp>
-      <kd>1.0</kd>
-      <mu1>100.0</mu1>
-      <mu2>100.0</mu2>
-      <maxVel>1.0</maxVel>
-      <minDepth>0.002</minDepth>
+      <mu1>0.9</mu1>
+      <mu2>0.9</mu2>
     </gazebo>
     <gazebo reference="fingertip1_1_link">
       <material>Gazebo/Grey</material>
       <self_collide>true</self_collide>
-      <kp>1000000.0</kp>
-      <kd>1.0</kd>
-      <mu1>100.0</mu1>
-      <mu2>100.0</mu2>
-      <maxVel>1.0</maxVel>
-      <minDepth>0.002</minDepth>
+      <mu1>0.9</mu1>
+      <mu2>0.9</mu2>
     </gazebo>
     <gazebo reference="fingertip1_2_link">
       <material>Gazebo/Grey</material>
       <self_collide>true</self_collide>
-      <kp>1000000.0</kp>
-      <kd>1.0</kd>
-      <mu1>100.0</mu1>
-      <mu2>100.0</mu2>
-      <maxVel>1.0</maxVel>
-      <minDepth>0.002</minDepth>
+      <mu1>0.9</mu1>
+      <mu2>0.9</mu2>
     </gazebo>
     <gazebo reference="fingertip2_1_link">
       <material>Gazebo/Grey</material>
       <self_collide>true</self_collide>
-      <kp>1000000.0</kp>
-      <kd>1.0</kd>
-      <mu1>100.0</mu1>
-      <mu2>100.0</mu2>
-      <maxVel>1.0</maxVel>
-      <minDepth>0.002</minDepth>
+      <mu1>0.9</mu1>
+      <mu2>0.9</mu2>
     </gazebo>
     <gazebo reference="fingertip2_2_link">
       <material>Gazebo/Grey</material>
       <self_collide>true</self_collide>
-      <kp>1000000.0</kp>
-      <kd>1.0</kd>
-      <mu1>100.0</mu1>
-      <mu2>100.0</mu2>
-      <maxVel>1.0</maxVel>
-      <minDepth>0.002</minDepth>
+      <mu1>0.9</mu1>
+      <mu2>0.9</mu2>
     </gazebo>
     </xacro:macro>
